File: RefleXion 65/RefleXion 65 - Matrix/RefleXion - Ortho 65.kicad_pcb (KiCad board)
At the start: 2 copper layers, 133.4 x 96.2 mm, 114 parts, among them J1 Conn_01x22, J2 Conn_01x01, J3 Conn_01x01, SW1 SW_Push, SW10 SW_Push, SW11 SW_Push, SW12 SW_Push, SW13 SW_Push, SW14 SW_Push, SW15 SW_Push, SW16 SW_Push, SW17 SW_Push, SW18 SW_Push, SW19 SW_Push, SW2 SW_Push, SW20 SW_Push, SW21 SW_Push, SW22 SW_Push, SW23 SW_Push, SW24 SW_Push, SW25 SW_Push, SW26 SW_Push, SW27 SW_Push, SW28 SW_Push, SW29 SW_Push, SW3 SW_Push, SW30 SW_Push, SW31 SW_Push, SW32 SW_Push, SW33 SW_Push, SW34 SW_Push, SW4 SW_Push, SW5 SW_Push, SW6 SW_Push, SW7 SW_Push, SW8 SW_Push, SW9 SW_Push

Commit message: big dump
Parts:
- removed J3: Conn_01x01, Connector_PinHeader_2.54mm:PinHeader_1x01_P2.54mm_Vertical
- removed the LED28 at (168.0, 109.7)
- removed the LED29 at (53.7, 128.7)
- removed the LED30 at (72.8, 128.7)
- removed the LED31 at (91.8, 128.7)
- removed the SW28 at (168.0, 104.6)
- removed the SW30 at (72.8, 123.7)
- added C10: 30pF, Capacitor_SMD:C_0402_1005Metric, F.Cu at (81.7, 70.6)
- added C11: 30pF, Capacitor_SMD:C_0402_1005Metric, F.Cu at (84.4, 70.0)
- added C12: 1uF, Capacitor_SMD:C_0402_1005Metric, F.Cu at (86.9, 51.9)
- added C13: 1uF, Capacitor_SMD:C_0402_1005Metric, F.Cu at (83.5, 53.6)
- added C14: 1uF, Capacitor_SMD:C_0402_1005Metric, F.Cu at (88.3, 55.4)
- added C15: 100nF, Capacitor_SMD:C_0402_1005Metric, F.Cu at (78.8, 61.4)
- added C16: 100nF, Capacitor_SMD:C_0402_1005Metric, F.Cu at (89.2, 56.9)
- added C17: 100nF, Capacitor_SMD:C_0402_1005Metric, F.Cu at (89.2, 57.8)
- added C18: 100nF, Capacitor_SMD:C_0402_1005Metric, F.Cu at (84.5, 66.3)
- added C19: 100nF, Capacitor_SMD:C_0402_1005Metric, F.Cu at (79.1, 58.0)
- added C20: 100nF, Capacitor_SMD:C_0402_1005Metric, F.Cu at (90.1, 61.3)
- added C21: 1uF, Capacitor_SMD:C_0402_1005Metric, F.Cu at (85.4, 66.3)
- added C22: 100nF, Capacitor_SMD:C_0402_1005Metric, F.Cu at (87.4, 55.4)
- added C23: 100nF, Capacitor_SMD:C_0402_1005Metric, F.Cu at (83.1, 55.0)
- added C5: 100nF, Capacitor_SMD:C_0603_1608Metric_Pad1.08x0.95mm_HandSolder, B.Cu at (73.4, 93.9)
- added C6: 100nF, Capacitor_SMD:C_0603_1608Metric_Pad1.08x0.95mm_HandSolder, B.Cu at (85.0, 94.0)
- added C7: 100nF, Capacitor_SMD:C_0603_1608Metric_Pad1.08x0.95mm_HandSolder, B.Cu at (73.3, 132.0)
- added C8: 100nF, Capacitor_SMD:C_0603_1608Metric_Pad1.08x0.95mm_HandSolder, B.Cu at (85.1, 132.1)
- added C9: 100nF, Capacitor_SMD:C_0402_1005Metric, F.Cu at (84.0, 55.0)
- added D35: 1N4148W, Diode_SMD:D_SOD-123, B.Cu at (146.8, 126.0)
- added D36: 1N4148W, Diode_SMD:D_SOD-123, B.Cu at (174.4, 115.4)
- added D37: 1N4148W, Diode_SMD:D_SOD-123, B.Cu at (193.4, 115.4)
- added D38: 1N4148W, Diode_SMD:D_SOD-123, B.Cu at (212.5, 115.4)
- added D40: 1N5819WS, Diode_SMD:D_SOD-323F, F.Cu at (83.1, 48.5)
- added ENC10: Rotary_Encoder_Click, Keyboard Encoders:Encoder_Alps_EC11E_Small, F.Cu at (79.1, 86.0)
- added ENC11: Rotary_Encoder_Click, Keyboard Encoders:Encoder_Alps_EC11E_Small, F.Cu at (79.1, 124.1)
- added ENC3: Rotary_Encoder_Click, Keyboard Encoders:Encoder_Alps_EC11E_Small, F.Cu at (212.5, 47.9)
- added ENC4: Rotary_Encoder_Click, Keyboard Encoders:Encoder_Alps_EC11E_Small, F.Cu at (174.4, 105.0)
- added ENC5: Rotary_Encoder_Click, Keyboard Encoders:Encoder_Alps_EC11E_Small, F.Cu at (193.4, 105.0)
- added ENC6: Rotary_Encoder_Click, Keyboard Encoders:Encoder_Alps_EC11E_Small, F.Cu at (212.5, 105.0)
- added ENC7: Rotary_Encoder_Click, Keyboard Encoders:Encoder_Alps_EC11E_Small, F.Cu at (174.4, 124.1)
- added ENC8: Rotary_Encoder_Click, Keyboard Encoders:Encoder_Alps_EC11E_Small, F.Cu at (193.4, 124.1)
- added ENC9: Rotary_Encoder_Click, Keyboard Encoders:Encoder_Alps_EC11E_Small, F.Cu at (212.5, 124.1)
- added F1: CF06V5TR50, Resistor_SMD:R_0603_1608Metric, F.Cu at (85.5, 47.7)
- added FB1: BLM18SG700TZ1D, Capacitor_SMD:C_0603_1608Metric_Pad1.08x0.95mm_HandSolder, F.Cu at (83.1, 46.8)
- added FB2: BLM18SG700TZ1D, Capacitor_SMD:C_0603_1608Metric_Pad1.08x0.95mm_HandSolder, F.Cu at (88.0, 40.0)
- added FB3: BLM18SG700TZ1D, Capacitor_SMD:C_0603_1608Metric_Pad1.08x0.95mm_HandSolder, F.Cu at (73.4, 56.2)
- added FB4: BLM18SG700TZ1D, Capacitor_SMD:C_0603_1608Metric_Pad1.08x0.95mm_HandSolder, F.Cu at (78.1, 69.5)
- added LED22: SK6812MINI-E, Keyboard RGB:MX_SK6812MINI-E_REVERSIBLE, F.Cu at (212.5, 91.0)
- added LED23: SK6812MINI-E, Keyboard RGB:MX_SK6812MINI-E_REVERSIBLE_special, F.Cu at (79.1, 110.1)
- added LED24: SK6812MINI-E, Keyboard RGB:MX_SK6812MINI-E_REVERSIBLE_special, F.Cu at (88.7, 99.0)
- added LED26: SK6812MINI-E, Keyboard RGB:MX_SK6812MINI-E_REVERSIBLE_special, F.Cu at (107.7, 99.7)
- added LED33: SK6812MINI-E, Keyboard RGB:MX_SK6812MINI-E_REVERSIBLE, F.Cu at (79.1, 129.1)
- added LED35: SK6812MINI-E, Keyboard RGB:MX_SK6812MINI-E_REVERSIBLE_special, F.Cu at (107.7, 119.0)
- added LED37: SK6812MINI-E, Keyboard RGB:MX_SK6812MINI-E_REVERSIBLE, F.Cu at (136.3, 129.1)
- added LED38: SK6812MINI-E, Keyboard RGB:MX_SK6812MINI-E_REVERSIBLE, F.Cu at (155.3, 129.1)
- added LED39: SK6812MINI-E, Keyboard RGB:MX_SK6812MINI-E_REVERSIBLE, F.Cu at (174.4, 129.1)
- added LED40: SK6812MINI-E, Keyboard RGB:MX_SK6812MINI-E_REVERSIBLE, F.Cu at (193.4, 129.1)
- added LED41: SK6812MINI-E, Keyboard RGB:MX_SK6812MINI-E_REVERSIBLE, F.Cu at (212.5, 129.1)
- added OLED1: OLED_4pin, Keyboard Common:SSD1306-0.91-OLED-4pin-128x32 doublesided, F.Cu at (80.9, 57.9)
- added R1: 10K, Resistor_SMD:R_0402_1005Metric, F.Cu at (73.5, 47.0)
- added R10: 68K, Resistor_SMD:R_0402_1005Metric, F.Cu at (89.0, 66.1)
- added R11: 68K, Resistor_SMD:R_0402_1005Metric, F.Cu at (89.0, 67.9)
- added R2: 1K, Resistor_SMD:R_0402_1005Metric, F.Cu at (73.5, 49.8)
- added R3: 27R, Resistor_SMD:R_0402_1005Metric, F.Cu at (85.2, 55.2)
- added R4: 27R, Resistor_SMD:R_0402_1005Metric, F.Cu at (86.1, 55.2)
- added R5: 10K, Resistor_SMD:R_0402_1005Metric, F.Cu at (81.1, 50.9)
- added R6: 1K, Resistor_SMD:R_0402_1005Metric, F.Cu at (84.4, 68.2)
- added R7: 5.1K, Resistor_SMD:R_0402_1005Metric, F.Cu at (81.0, 47.6)
- added R8: 5.1K, Resistor_SMD:R_0402_1005Metric, F.Cu at (76.5, 47.6)
- added R9: 68K, Resistor_SMD:R_0402_1005Metric, F.Cu at (88.0, 66.1)
- added ST2: Stabilizer_2u_MX, Keyboard Stabilizer:Stabilizer_Cherry_MX_2.00u, F.Cu at (-25.7, 81.1)
- added ST3: Stabilizer_2u_MX, Keyboard Stabilizer:Stabilizer_Cherry_MX_2.00u, F.Cu at (-25.7, 101.9)
- added SW23: SW_Push, Keyboard Switches:SW_MX_HotSwap_Reversible, F.Cu at (79.1, 105.0)
- added SW24: SW_Push, Keyboard Switches:SW_MX_HotSwap_Reversible, F.Cu at (88.7, 105.0)
- added SW26: SW_Push, Keyboard Switches:SW_MX_HotSwap_Reversible, F.Cu at (107.7, 105.8)
- added SW31: SW_Push, Keyboard Switches:SW_MX_HotSwap_Reversible, F.Cu at (193.4, 105.0)
- added SW32: SW_Push, Keyboard Switches:SW_MX_HotSwap_Reversible, F.Cu at (212.5, 105.0)
- added SW33: SW_Push, Keyboard Switches:SW_MX_HotSwap_Reversible, F.Cu at (79.1, 124.1)
- added SW35: SW_Push, Keyboard Switches:SW_MX_HotSwap_Reversible, F.Cu at (107.7, 124.1)
- added SW39: SW_Push, Keyboard Switches:SW_MX_HotSwap_Reversible, F.Cu at (174.4, 124.1)
- added SW41: SW_Push, Keyboard Switches:SW_MX_HotSwap_Reversible, F.Cu at (212.5, 124.1)
- added SW42: YTSA010, Keyboard Common:YTS-A002, F.Cu at (71.0, 44.1)
- added SW43: YTSA010, Keyboard Common:YTS-A002, F.Cu at (70.9, 51.3)
- added U1: W25Q32JVUUIQ, Keyboard Common:USON-8_4x3mm_P0.8mm, F.Cu at (80.0, 54.2)
- added U2: RP2040, Package_DFN_QFN:QFN-56-1EP_7x7mm_P0.4mm_EP3.2x3.2mm, F.Cu at (84.1, 60.9)
- added U3: SRV05-4, Package_TO_SOT_SMD:SOT-23-6_Handsoldering, F.Cu at (78.7, 49.1)
- added U4: SPX3819M5-L-3-3/TR, Package_TO_SOT_SMD:SOT-23-5, F.Cu at (83.9, 51.2)
- added U6: SN74LV1T34DBV, Package_TO_SOT_SMD:SOT-23-5, F.Cu at (88.4, 49.7)
- added Y1: TXM12M0004252LBCEO00T, Crystal:Crystal_SMD_2520-4Pin_2.5x2.0mm, F.Cu at (82.2, 68.6)
- ENC1: renamed from ENC2; footprint Keyboard Encoders:Encoder_Alps_EC11E_Offset_pad -> Keyboard Encoders:Encoder_Alps_EC11E_Small
- ENC2: renamed from ENC1; footprint Keyboard Encoders:Encoder_Alps_EC11E_Offset_pad -> Keyboard Encoders:Encoder_Alps_EC11E_Small
- J1: value Conn_01x22 -> USB_C_Receptacle_USB2.0; footprint Connector_PinHeader_2.54mm:PinHeader_1x22_P2.54mm_Vertical -> Keyboard Common:Molex-216990_GCT-USB45xx_HRO-TYPE-C-31-M-13x-PiMicro
- J2: value Conn_01x01 -> USB_C_Receptacle_USB2.0; footprint Connector_PinHeader_2.54mm:PinHeader_1x01_P2.54mm_Vertical -> Keyboard Common:Molex-216990_GCT-USB45xx_HRO-TYPE-C-31-M-13x-PiMicro
- LED25: renamed from LED27; footprint Keyboard RGB:MX_SK6812MINI-E_REVERSIBLE -> Keyboard RGB:MX_SK6812MINI-E_REVERSIBLE_special
- LED27: renamed from LED26; footprint Keyboard RGB:MX_SK6812MINI-E_REVERSIBLE -> Keyboard RGB:MX_SK6812MINI-E_REVERSIBLE_special
- LED34: footprint Keyboard RGB:MX_SK6812MINI-E_REVERSIBLE -> Keyboard RGB:MX_SK6812MINI-E_REVERSIBLE_special
- LED36: renamed from LED33; footprint Keyboard RGB:MX_SK6812MINI-E_REVERSIBLE -> Keyboard RGB:MX_SK6812MINI-E_REVERSIBLE_special
- Logo1: footprint Logotypes:CC_BY_SA_40 -> Logotypes:CC_BY_SA_40_line; moved to F.Cu
- moved ST1 194.8 mm to (-25.7, 60.4), turned to 0 degrees
- moved D22 164.2 mm to (212.5, 77.0), turned to 180 degrees
- moved SW22 159.8 mm to (212.5, 86.0)
- moved D30 150.6 mm to (211.4, 95.6), turned to 180 degrees
- moved D29 144.5 mm to (192.3, 95.6), turned to 180 degrees
- moved ENC2 139.7 mm to (193.4, 47.9)
- moved LED13 139.7 mm to (193.4, 72.0)
- moved LED21 139.7 mm to (193.4, 91.0)
- moved LED31 139.7 mm to (193.4, 110.1)
- moved LED6 139.7 mm to (193.4, 52.9)
- moved SW13 139.7 mm to (193.4, 66.9)
- moved SW21 139.7 mm to (193.4, 86.0)
- moved SW40 139.7 mm to (193.4, 124.1)
- moved SW6 139.7 mm to (193.4, 47.9)
- moved C4 135.5 mm to (180.4, 113.0), turned to 180 degrees
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- renumbered LED6 to LED1, LED11 to LED10, LED10 to LED11, LED9 to LED12, LED8 to LED13, LED21 to LED15, LED20 to LED16, LED19 to LED17, LED17 to LED19, LED5 to LED2, LED16 to LED20, LED15 to LED21, LED25 to LED28, LED24 to LED29, LED4 to LED3, LED23 to LED30, LED22 to LED31, LED3 to LED4, LED2 to LED5, LED1 to LED6, LED13 to LED8, LED12 to LED9, SW6 to SW1, SW11 to SW10, SW10 to SW11, SW9 to SW12, SW8 to SW13, SW21 to SW15, SW20 to SW16, SW19 to SW17, SW17 to SW19, SW5 to SW2, SW16 to SW20, SW15 to SW21, SW27 to SW25, SW26 to SW27, SW25 to SW28, SW24 to SW29, SW4 to SW3, SW23 to SW30, SW33 to SW36, SW32 to SW37, SW31 to SW38, SW3 to SW4, SW29 to SW40, SW2 to SW5, SW1 to SW6, SW13 to SW8, SW12 to SW9
Connections:
- C1 pad 1: B1 -> EncA
- C2 pad 2: A2 -> EncB
- C3 pad 1: A1 -> EncB
- C4 pad 2: B1 -> EncC
- D1 pad 2: Enc1 -> Net-(D1-A)
- D10 pad 2: Net-(D10-Pad2) -> Net-(D10-A)
- D11 pad 2: Net-(D11-Pad2) -> Net-(D11-A)
- D12 pad 2: Net-(D12-Pad2) -> Net-(D12-A)
- D13 pad 2: Net-(D13-Pad2) -> Net-(D13-A)
- D15 pad 2: Net-(D15-Pad2) -> Enc10
- D16 pad 2: Net-(D16-Pad2) -> Net-(D16-A)
- D17 pad 2: Net-(D17-Pad2) -> Net-(D17-A)
- D19 pad 2: Net-(D19-Pad2) -> Net-(D19-A)
- D2 pad 2: Net-(D2-Pad2) -> Net-(D2-A)
- D20 pad 2: Net-(D20-Pad2) -> Net-(D20-A)
- D21 pad 2: Net-(D21-Pad2) -> Net-(D21-A)
- D22 pad 1: Row3 -> Row2
- D23 pad 2: Net-(D23-Pad2) -> Net-(D23-A)
- D24 pad 2: Net-(D24-Pad2) -> Net-(D24-A)
- D25 pad 2: Net-(D25-Pad2) -> Net-(D25-A)
- D26 pad 2: Net-(D26-Pad2) -> Net-(D26-A)
- D27 pad 2: Net-(D27-Pad2) -> Net-(D27-A)
- D28 pad 2: Net-(D28-Pad2) -> Enc4
- D29 pad 1: Row4 -> Row3
- D29 pad 2: Net-(D29-Pad2) -> Enc5
- D3 pad 2: Net-(D3-Pad2) -> Net-(D3-A)
- D30 pad 1: Row4 -> Row3
- D30 pad 2: Net-(D30-Pad2) -> Enc6
- D31 pad 2: Net-(D31-Pad2) -> Enc11
- D32 pad 2: Net-(D32-Pad2) -> Net-(D32-A)
- D34 pad 2: Net-(D34-Pad2) -> Net-(D34-A)
- D4 pad 2: Net-(D4-Pad2) -> Net-(D4-A)
- D5 pad 2: Net-(D5-Pad2) -> Enc1
- D6 pad 2: Net-(D6-Pad2) -> Enc2
- D7 pad 2: Enc2 -> Enc3
- D8 pad 2: Net-(D8-Pad2) -> Net-(D8-A)
- D9 pad 2: Net-(D9-Pad2) -> Net-(D9-A)
- ENC1 pad A: B1 -> EncA
- ENC1 pad B: A2 -> EncB
- ENC1 pad S1: Col6 -> Col5
- ENC1 pad S2: Enc2 -> Enc1
- ENC2 pad A: A1 -> EncA
- ENC2 pad B: B1 -> EncB
- ENC2 pad S1: Col0 -> Col6
- ENC2 pad S2: Enc1 -> Enc2
- LED1 pad 1: VCC -> +5V
- LED1 pad 2: Net-(LED6-Pad2) -> Net-(LED1-DOUT)
- LED1 pad 4: Net-(LED5-Pad2) -> Net-(LED1-DIN)
- LED10 pad 1: VCC -> +5V
- LED10 pad 2: Net-(LED10-Pad4) -> Net-(LED10-DOUT)
- LED10 pad 4: Net-(LED11-Pad4) -> Net-(LED10-DIN)
- LED11 pad 1: VCC -> +5V
- LED11 pad 2: Net-(LED10-Pad2) -> Net-(LED10-DIN)
- LED11 pad 4: Net-(LED10-Pad4) -> Net-(LED11-DIN)
- LED12 pad 1: VCC -> +5V
- LED12 pad 2: Net-(LED8-Pad4) -> Net-(LED11-DIN)
- LED12 pad 4: Net-(LED10-Pad2) -> Net-(LED12-DIN)
- LED13 pad 1: VCC -> +5V
- LED13 pad 2: Net-(LED15-Pad4) -> Net-(LED12-DIN)
- LED13 pad 4: Net-(LED8-Pad4) -> Net-(LED13-DIN)
- LED14 pad 1: VCC -> +5V
- LED14 pad 2: Net-(LED13-Pad4) -> Net-(LED13-DIN)
- LED15 pad 1: VCC -> +5V
- LED15 pad 2: Net-(LED21-Pad2) -> Net-(LED15-DOUT)
- LED15 pad 4: Net-(LED20-Pad2) -> Net-(LED15-DIN)
- LED16 pad 1: VCC -> +5V
- LED16 pad 2: Net-(LED20-Pad2) -> Net-(LED16-DOUT)
- LED16 pad 4: Net-(LED19-Pad2) -> Net-(LED15-DOUT)
- LED17 pad 1: VCC -> +5V
- LED17 pad 2: Net-(LED19-Pad2) -> Net-(LED17-DOUT)
- LED17 pad 4: Net-(LED18-Pad2) -> Net-(LED16-DOUT)
- LED18 pad 1: VCC -> +5V
- LED18 pad 2: Net-(LED18-Pad2) -> Net-(LED18-DOUT)
- LED18 pad 4: Net-(LED17-Pad2) -> Net-(LED17-DOUT)
- LED19 pad 1: VCC -> +5V
- LED19 pad 2: Net-(LED17-Pad2) -> Net-(LED19-DOUT)
- LED19 pad 4: Net-(LED16-Pad2) -> Net-(LED18-DOUT)
- LED2 pad 1: VCC -> +5V
- LED2 pad 2: Net-(LED5-Pad2) -> Net-(LED2-DOUT)
- LED2 pad 4: Net-(LED4-Pad2) -> Net-(LED1-DOUT)
- LED20 pad 1: VCC -> +5V
- LED20 pad 2: Net-(LED16-Pad2) -> Net-(LED20-DOUT)
- LED20 pad 4: Net-(LED15-Pad2) -> Net-(LED19-DOUT)
- LED21 pad 1: VCC -> +5V
- LED21 pad 2: Net-(LED15-Pad2) -> Net-(LED21-DOUT)
- LED21 pad 4: Net-(LED15-Pad4) -> Net-(LED20-DOUT)
- LED25 pad 1: VCC -> +5V
- LED25 pad 2: Net-(LED26-Pad4) -> Net-(LED24-DIN)
- LED27 pad 1: VCC -> +5V
- LED27 pad 2: Net-(LED25-Pad4) -> Net-(LED26-DIN)
- LED27 pad 4: Net-(LED26-Pad4) -> Net-(LED27-DIN)
- LED28 pad 1: VCC -> +5V
- LED28 pad 2: Net-(LED24-Pad4) -> Net-(LED27-DIN)
- LED28 pad 4: Net-(LED25-Pad4) -> Net-(LED28-DIN)
- LED29 pad 1: VCC -> +5V
- LED29 pad 2: Net-(LED23-Pad4) -> Net-(LED28-DIN)
- LED29 pad 4: Net-(LED24-Pad4) -> Net-(LED29-DIN)
- LED3 pad 1: VCC -> +5V
- LED3 pad 2: Net-(LED4-Pad2) -> Net-(LED3-DOUT)
- LED3 pad 4: Net-(LED3-Pad2) -> Net-(LED2-DOUT)
- LED30 pad 1: VCC -> +5V
- LED30 pad 2: Net-(LED22-Pad4) -> Net-(LED29-DIN)
- LED30 pad 4: Net-(LED23-Pad4) -> Net-(LED30-DIN)
- LED31 pad 1: VCC -> +5V
- LED31 pad 2: Net-(LED22-Pad2) -> Net-(LED30-DIN)
- LED31 pad 4: Net-(LED22-Pad4) -> Net-(LED31-DIN)
- LED32 pad 1: VCC -> +5V
- LED32 pad 2: Net-(LED32-Pad2) -> Net-(LED31-DIN)
- LED34 pad 1: VCC -> +5V
- LED34 pad 2: unconnected-(LED34-Pad2) -> Net-(LED34-DOUT)
- LED34 pad 4: Net-(LED33-Pad2) -> Net-(LED33-DOUT)
- LED36 pad 1: VCC -> +5V
- LED36 pad 2: Net-(LED33-Pad2) -> Net-(LED36-DOUT)
- LED36 pad 4: Net-(LED32-Pad2) -> Net-(LED35-DOUT)
- LED4 pad 1: VCC -> +5V
- LED4 pad 2: Net-(LED3-Pad2) -> Net-(LED4-DOUT)
- LED4 pad 4: Net-(LED2-Pad2) -> Net-(LED3-DOUT)
- LED5 pad 1: VCC -> +5V
- LED5 pad 2: Net-(LED2-Pad2) -> Net-(LED5-DOUT)
- LED5 pad 4: Net-(LED1-Pad2) -> Net-(LED4-DOUT)
- LED6 pad 1: VCC -> +5V
- LED6 pad 2: Net-(LED1-Pad2) -> Net-(LED6-DOUT)
- LED6 pad 4: RGB -> Net-(LED5-DOUT)
- LED7 pad 1: VCC -> +5V
- LED7 pad 4: Net-(LED6-Pad2) -> Net-(LED6-DOUT)
- LED8 pad 1: VCC -> +5V
- LED8 pad 2: Net-(LED12-Pad4) -> Net-(LED15-DIN)
- LED8 pad 4: Net-(LED13-Pad4) -> Net-(LED8-DIN)
- LED9 pad 1: VCC -> +5V
- LED9 pad 2: Net-(LED11-Pad4) -> Net-(LED8-DIN)
- LED9 pad 4: Net-(LED12-Pad4) -> Net-(LED10-DOUT)
- SW1 pad 1: Net-(D6-Pad2) -> Net-(D1-A)
- SW1 pad 2: Col5 -> Col1
- SW10 pad 1: Net-(D11-Pad2) -> Net-(D10-A)
- SW11 pad 1: Net-(D10-Pad2) -> Net-(D11-A)
- SW11 pad 2: Col2 -> Col4
- SW12 pad 1: Net-(D9-Pad2) -> Net-(D12-A)
- SW12 pad 2: Col1 -> Col5
- SW13 pad 1: Net-(D8-Pad2) -> Net-(D13-A)
- SW13 pad 2: Col0 -> Col6
- SW14 pad 2: Col6 -> Col7
- SW15 pad 1: Net-(D21-Pad2) -> Enc10
- SW15 pad 2: Col6 -> Col0
- SW16 pad 1: Net-(D20-Pad2) -> Net-(D16-A)
- SW16 pad 2: Col5 -> Col1
- SW17 pad 1: Net-(D19-Pad2) -> Net-(D17-A)
- SW17 pad 2: Col4 -> Col2
- SW19 pad 1: Net-(D17-Pad2) -> Net-(D19-A)
- SW19 pad 2: Col2 -> Col4
- SW2 pad 1: Net-(D5-Pad2) -> Net-(D2-A)
- SW2 pad 2: Col4 -> Col2
- SW20 pad 1: Net-(D16-Pad2) -> Net-(D20-A)
- SW20 pad 2: Col1 -> Col5
- SW21 pad 1: Net-(D15-Pad2) -> Net-(D21-A)
- SW21 pad 2: Col0 -> Col6
- SW22 pad 2: Col0 -> Col7
- SW25 pad 1: Net-(D27-Pad2) -> Net-(D24-A)
- SW25 pad 2: Col5 -> Col1
- SW27 pad 1: Net-(D26-Pad2) -> Net-(D25-A)
- SW27 pad 2: Col4 -> Col2
- SW28 pad 1: Net-(D25-Pad2) -> Net-(D26-A)
- SW29 pad 1: Net-(D24-Pad2) -> Net-(D27-A)
- SW29 pad 2: Col2 -> Col4
- SW3 pad 1: Net-(D4-Pad2) -> Net-(D3-A)
- SW30 pad 1: Net-(D23-Pad2) -> Enc4
- SW30 pad 2: Col1 -> Col5
- SW34 pad 1: Net-(D34-Pad2) -> Col1
- SW34 pad 2: Col5 -> Net-(D32-A)
- SW36 pad 2: Col4 -> Col2
- SW37 pad 1: Net-(D32-Pad2) -> Net-(D34-A)
- SW38 pad 1: Net-(D31-Pad2) -> Net-(D35-A)
- SW38 pad 2: Col2 -> Col4
- SW4 pad 1: Net-(D3-Pad2) -> Net-(D4-A)
- SW4 pad 2: Col2 -> Col4
- SW40 pad 1: Net-(D29-Pad2) -> Enc8
- SW40 pad 2: Col0 -> Col6
- SW5 pad 1: Net-(D2-Pad2) -> Enc1
- SW5 pad 2: Col1 -> Col5
- SW6 pad 1: Enc1 -> Enc2
- SW6 pad 2: Col0 -> Col6
- SW7 pad 1: Enc2 -> Enc3
- SW7 pad 2: Col6 -> Col7
- SW8 pad 1: Net-(D13-Pad2) -> Net-(D8-A)
- SW8 pad 2: Col5 -> Col1
- SW9 pad 1: Net-(D12-Pad2) -> Net-(D9-A)
- SW9 pad 2: Col4 -> Col2
Routing:
- net +5V: track 0.00 -> 1084.8 mm, vias 0 -> 70
- net VCC: track 784.0 -> 0.00 mm, vias 40 -> 0
- net EncB: track 0.00 -> 367.1 mm, vias 0 -> 10
- net EncC: track 0.00 -> 352.3 mm, vias 0 -> 15
- net Col7: track 0.00 -> 243.2 mm, vias 0 -> 7
- net GND: track 109.6 -> 294.8 mm, vias 43 -> 129
- net EncA: track 0.00 -> 166.5 mm, vias 0 -> 6
- net B1: track 134.5 -> 0.00 mm, vias 1 -> 0
- net Col6: track 115.4 -> 224.3 mm
- net A2: track 98.0 -> 0.00 mm, vias 1 -> 0
- net EncD: track 0.00 -> 90.6 mm, vias 0 -> 2
- net Col5: track 123.3 -> 204.9 mm, vias 10 -> 7
- net +3V3: track 0.00 -> 59.8 mm, vias 0 -> 4
- net Col1: track 87.7 -> 147.2 mm, vias 10 -> 9
- net Col3: track 86.9 -> 143.1 mm, vias 10 -> 6
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Other:
- board size 133.4 x 96.2 mm -> 152.4 x 95.2 mm
- board text added: "Design: Markus Knutsson Concept: Pedro Quaresma"
- board text added: "RefleXion 65 - 2023 - https://github.com/TweetyDaBird Licensed under Creative Commons BY-SA 4.0 International"
- board text removed: "Design: Markus Knutsson - Concept: Pedro Quaresma"
- board text removed: "Licensed under Creative Commons BY-SA 4.0 International"
- board text removed: "RefleXion - Ortho 65 Matrix - 2022"
- board text removed: "https://github.com/TweetyDaBird"
