File: RefleXion 65/RefleXion 65 - Matrix/RefleXion - Ortho 65.kicad_sch (KiCad schematic)
At the start: 118 parts, among them J1 Conn_01x22, J2 Conn_01x01, J3 Conn_01x01, SW1 SW_Push, SW10 SW_Push, SW11 SW_Push, SW12 SW_Push, SW13 SW_Push, SW14 SW_Push, SW15 SW_Push, SW16 SW_Push, SW17 SW_Push, SW18 SW_Push, SW19 SW_Push, SW2 SW_Push, SW20 SW_Push, SW21 SW_Push, SW22 SW_Push, SW23 SW_Push, SW24 SW_Push, SW25 SW_Push, SW26 SW_Push, SW27 SW_Push, SW28 SW_Push, SW29 SW_Push, SW3 SW_Push, SW30 SW_Push, SW31 SW_Push, SW32 SW_Push, SW33 SW_Push, SW34 SW_Push, SW4 SW_Push, SW5 SW_Push, SW6 SW_Push, SW7 SW_Push, SW8 SW_Push, SW9 SW_Push

Commit message: big dump
Parts:
- removed C1: 100nF, Capacitor_SMD:C_0603_1608Metric_Pad1.08x0.95mm_HandSolder, symbol Device:C_Small
- removed H1, H2, H3, H4: Spacer_PCB, Keyboard Common:Spacer PCB hole, symbol Keyboard_Plate:Spacer_PCB
- removed J1: Conn_01x22, Connector_PinHeader_2.54mm:PinHeader_1x22_P2.54mm_Vertical, symbol Connector_Generic:Conn_01x22
- removed J2, J3: Conn_01x01, Connector_PinHeader_2.54mm:PinHeader_1x01_P2.54mm_Vertical, symbol Connector_Generic:Conn_01x01
- added C10, C11: 30pF, Capacitor_SMD:C_0402_1005Metric, symbol Device:C
- added C12, C13, C14, C21: 1uF, Capacitor_SMD:C_0402_1005Metric, symbol Device:C
- added C15, C16, C17, C18, C19, C20, C22, C23, C9: 100nF, Capacitor_SMD:C_0402_1005Metric, symbol Device:C
- added C4, C5, C6, C7, C8: 100nF, Capacitor_SMD:C_0603_1608Metric_Pad1.08x0.95mm_HandSolder, symbol Device:C_Small
- added D22, D30, D37, D38: 1N4148W, Diode_SMD:D_SOD-123, symbol Diode:1N4148W
- added D40: 1N5819WS, Diode_SMD:D_SOD-323F, symbol Device:D_Schottky_Small
- added ENC10, ENC11, ENC3, ENC4, ENC5, ENC6, ENC7, ENC8, ENC9: Rotary_Encoder_Click, Keyboard Encoders:Encoder_Alps_EC11E_Small, symbol Keyboard Switches:Rotary_Encoder_Click
- added F1: CF06V5TR50, Resistor_SMD:R_0603_1608Metric, symbol Device:Polyfuse_Small
- added FB1, FB2, FB3, FB4: BLM18SG700TZ1D, Capacitor_SMD:C_0603_1608Metric_Pad1.08x0.95mm_HandSolder, symbol LCSC Parts:Ferrite Bead
- added J1, J2: USB_C_Receptacle_USB2.0, Keyboard Common:Molex-216990_GCT-USB45xx_HRO-TYPE-C-31-M-13x-PiMicro, symbol Connector:USB_C_Receptacle_USB2.0
- added LED35, LED36: SK6812MINI-E, Keyboard RGB:MX_SK6812MINI-E_REVERSIBLE_special, symbol Keyboard Common:SK6812MINI-E
- added LED37, LED38, LED39, LED40, LED41: SK6812MINI-E, Keyboard RGB:MX_SK6812MINI-E_REVERSIBLE, symbol Keyboard Common:SK6812MINI-E
- added OLED1: OLED_4pin, Keyboard Common:SSD1306-0.91-OLED-4pin-128x32 doublesided, symbol Keyboard Common:OLED_4pin
- added R1, R5: 10K, Resistor_SMD:R_0402_1005Metric, symbol Device:R
- added R10, R11, R9: 68K, Resistor_SMD:R_0402_1005Metric, symbol Device:R_Small
- added R2, R6: 1K, Resistor_SMD:R_0402_1005Metric, symbol Device:R
- added R3, R4: 27R, Resistor_SMD:R_0402_1005Metric, symbol Device:R_Small
- added R7, R8: 5.1K, Resistor_SMD:R_0402_1005Metric, symbol Device:R_Small
- added ST2, ST3: Stabilizer_2u_MX, Keyboard Stabilizer:Stabilizer_Cherry_MX_2.00u, symbol Keyboard Switches:Stabilizer_2u_MX
- added SW22, SW23, SW25, SW32, SW34, SW40, SW41: SW_Push, Keyboard Switches:SW_MX_HotSwap_Reversible, symbol Keyboard Switches:SW_MX_HotSwap_Reversible
- added SW42, SW43: YTSA010, Keyboard Common:YTS-A002, symbol Keyboard Common:TS-A002
- added U1: W25Q32JVUUIQ, Keyboard Common:USON-8_4x3mm_P0.8mm, symbol Memory_Flash:W25Q32JVSS
- added U2: RP2040, Package_DFN_QFN:QFN-56-1EP_7x7mm_P0.4mm_EP3.2x3.2mm, symbol MCU_RaspberryPi:RP2040
- added U3: SRV05-4, Package_TO_SOT_SMD:SOT-23-6_Handsoldering, symbol LCSC Parts:SRV05-4
- added U4: SPX3819M5-L-3-3/TR, Package_TO_SOT_SMD:SOT-23-5, symbol Regulator_Linear:SPX3819M5-L-3-3
- added U6: SN74LV1T34DBV, Package_TO_SOT_SMD:SOT-23-5, symbol Logic_LevelTranslator:SN74LV1T34DBV
- added Y1: TXM12M0004252LBCEO00T, Crystal:Crystal_SMD_2520-4Pin_2.5x2.0mm, symbol Device:Crystal_GND24
- ENC1, ENC2: footprint Keyboard Encoders:Encoder_Alps_EC11E_Offset_pad -> Keyboard Encoders:Encoder_Alps_EC11E_Small
- LED23, LED24, LED25, LED26, LED27, LED34: footprint Keyboard RGB:MX_SK6812MINI-E_REVERSIBLE -> Keyboard RGB:MX_SK6812MINI-E_REVERSIBLE_special
- Logo1: footprint Logotypes:CC_BY_SA_40 -> Logotypes:CC_BY_SA_40_line
- renumbered C3 to C1, C4 to C3, D22 to D23, D23 to D24, D24 to D25, D25 to D26, D26 to D27, D27 to D28, D28 to D29, D29 to D31, D30 to D32, D31 to D33, D32 to D34, D33 to D35, D34 to D36, SW22 to SW24, SW23 to SW26, SW24 to SW27, SW25 to SW28, SW26 to SW29, SW27 to SW30, SW28 to SW31, SW29 to SW33, SW30 to SW35, SW31 to SW36, SW32 to SW37, SW33 to SW38, SW34 to SW39
Connections:
- net Col0: now also ENC10.S1, ENC11.S1, SW23.2, U2.15 (GPIO12); no longer ENC1.S1, SW1.2, SW8.2
- net Col1: now also SW1.2, SW8.2, SW25.2, SW34.1, U2.32 (GPIO21); no longer SW2.2, SW9.2
- net Col2: now also SW2.2, SW9.2, U2.35 (GPIO23); no longer SW10.2, SW3.2
- net Col3: now also SW10.2, SW3.2, U2.36 (GPIO24); no longer SW11.2, SW4.2
- net Col4: now also SW11.2, SW4.2, U2.37 (GPIO25); no longer SW12.2, SW5.2
- net Col5: now also ENC1.S1, SW12.2, SW5.2, ENC4.S1, ENC7.S1, U2.38 (GPIO26_ADC0); no longer SW13.2, SW6.2
- net Col6: now also SW13.2, SW6.2, ENC5.S1, ENC8.S1, SW40.2, U2.39 (GPIO27_ADC1); no longer SW14.2, SW7.2
- net Enc1: now also D5.2 (A), SW5.1; no longer D1.2 (A), SW1.1
- net Enc2: now also D6.2 (A), SW6.1; no longer D7.2 (A), SW7.1
- net GND: now also C3.2, C10.2, C11.2, C12.2, C13.2, C14.2, C15.2, C16.2, C17.2, C18.2, C19.2, C20.2, C21.2, C22.2, C23.2, C4.1, C5.2, C6.1, C7.2, C8.1, C9.2, ENC10.C, ENC10.MP1 (GND), ENC10.MP2 (GND), ENC11.C, ENC11.MP1 (GND), ENC11.MP2 (GND), ENC3.C, ENC3.MP1 (GND), ENC3.MP2 (GND), ENC4.C, ENC4.MP1 (GND), ENC4.MP2 (GND), ENC5.C, ENC5.MP1 (GND), ENC5.MP2 (GND), ENC6.C, ENC6.MP1 (GND), ENC6.MP2 (GND), ENC7.C, ENC7.MP1 (GND), ENC7.MP2 (GND), ENC8.C, ENC8.MP1 (GND), ENC8.MP2 (GND), ENC9.C, ENC9.MP1 (GND), ENC9.MP2 (GND), FB2.2, FB3.2, J1.A1 (GND), J1.A12 (GND), J1.B1 (GND), J1.B12 (GND), J2.A1 (GND), J2.A12 (GND), J2.B1 (GND), J2.B12 (GND), LED35.3 (GND), LED36.3 (GND), LED37.3 (GND), LED38.3 (GND), LED39.3 (GND), LED40.3 (GND), LED41.3 (GND), OLED1.1 (GND), R11.2, R7.1, R8.2, SW42.1, SW42.3, SW43.1, SW43.3, U1.4 (GND), U2.19 (TESTEN), U2.57 (GND), U3.2 (VN), U4.2 (GND), U6.3 (GND), Y1.2, Y1.4; no longer C3.1
- net RGB: now also U2.31 (GPIO20), U6.2 (A); no longer LED1.4 (DIN)
- net Row0: now also U2.41 (GPIO29_ADC3)
- net Row1: now also U2.34 (GPIO22)
- net Row2: now also D22.1 (K), U2.29 (GPIO18)
- net Row3: now also D30.1 (K), U2.16 (GPIO13)
- net Row4: now also D37.1 (K), D38.1 (K), U2.14 (GPIO11)
- net SCL: now also OLED1.3 (SCL), U2.28 (GPIO17)
- net SDA: now also OLED1.4 (SDA), U2.27 (GPIO16)
- net at LED33.4 (DIN): now also LED23.2 (DOUT); no longer LED32.2 (DOUT)
- net Enc11: now reaches D31.2 (A), SW33.1
- net Enc11: now also ENC11.S2
- net at LED31.2 (DOUT): now also LED30.4 (DIN); no longer LED32.4 (DIN)
- net at LED31.4 (DIN): now also LED32.2 (DOUT); no longer LED30.2 (DOUT)
- net at LED22.4 (DIN): now also LED21.2 (DOUT); no longer LED23.2 (DOUT)
- net at LED28.4 (DIN): now also LED29.2 (DOUT); no longer LED21.2 (DOUT)
- net Enc5: now reaches D29.2 (A), SW31.1
- net Enc5: now also ENC5.S2
- net at LED34.2 (DOUT): now also LED35.4 (DIN)
- net Enc10: now reaches D15.2 (A), SW15.1
- net Enc10: now also ENC10.S2
- net at D24.2 (A), SW26.1: now also SW25.1
- net at D23.2 (A), SW24.1: now also SW23.1
- net at D32.2 (A), SW35.1: now also SW34.2
- net Enc4: now reaches D28.2 (A), SW30.1
- net Enc4: now also ENC4.S2
- net at LED29.4 (DIN): now also LED30.2 (DOUT); no longer LED22.2 (DOUT)
- net Enc7: now reaches D36.2 (A), SW39.1
- net Enc7: now also ENC7.S2
- net A1 renamed EncA
- net EncA: now also ENC2.A, ENC3.A, U2.17 (GPIO14)
- net A2 renamed EncB
- net EncB: now also C3.1, ENC1.B, ENC3.B, ENC4.A, ENC5.A, ENC6.A, ENC7.A, ENC8.A, ENC9.A, U2.18 (GPIO15)
- removed net B1: C3.2, ENC1.B, ENC2.A
- net VCC renamed +5V
- net +5V: now also C12.1, F1.2, FB4.2, LED35.1 (VDD), LED36.1 (VDD), LED37.1 (VDD), LED38.1 (VDD), LED39.1 (VDD), LED40.1 (VDD), LED41.1 (VDD), OLED1.2 (VCC), U4.1 (IN), U4.3 (EN), U6.5 (VCC)
- new net: LED39.2 (DOUT), LED40.4 (DIN)
- new net: LED38.2 (DOUT), LED39.4 (DIN)
- new net: D40.1 (K), F1.1
- new net: D1.2 (A), SW1.1
- new net: FB1.1, J1.A4 (VBUS), J1.A9 (VBUS), J1.B4 (VBUS), J1.B9 (VBUS)
- new net: J1.A5 (CC1), R7.2
- new net: J1.B5 (CC2), R8.1
- new net: R6.1, U2.21 (XOUT)
- new net: C11.1, R6.2, Y1.3
- new net: C10.1, U2.20 (XIN), Y1.1
- new net: FB4.1, J2.A4 (VBUS), J2.A9 (VBUS), J2.B4 (VBUS), J2.B9 (VBUS)
- new net: D22.2 (A), SW22.1
- new net: LED22.2 (DOUT), LED32.4 (DIN)
- new net: LED40.2 (DOUT), LED41.4 (DIN)
- new net: LED36.2 (DOUT), LED37.4 (DIN)
- new net: LED35.2 (DOUT), LED36.4 (DIN)
- new net: R2.2, SW43.2
- new net: R1.2, SW42.2, U2.26 (RUN)
- new net: U1.7 (IO3), U2.51 (QSPI_SD3)
- new net: U1.6 (CLK), U2.52 (QSPI_SCLK)
- new net: U1.5 (DI(IO0)), U2.53 (QSPI_SD0)
- new net: U1.3 (IO2), U2.54 (QSPI_SD2)
- new net: U1.2 (DO(IO1)), U2.55 (QSPI_SD1)
- new net: R2.1, R5.2, U1.1 (~{CS}), U2.56 (QSPI_SS)
- new net: OLED1.A (0), OLED1.B (0), OLED1.C (0), OLED1.D (0)
- new net: LED37.2 (DOUT), LED38.4 (DIN)
- new net: LED1.4 (DIN), U6.4 (Y)
- new net: R10.2, R11.1
- new net +1V1: C21.1, C22.1, C23.1, U2.23 (DVDD), U2.45 (VREG_VOUT), U2.50 (DVDD)
- new net +3V3: C13.1, C14.1, C15.1, C16.1, C17.1, C18.1, C19.1, C20.1, C9.1, R1.1, R5.1, U1.8 (VCC), U2.1 (IOVDD), U2.10 (IOVDD), U2.22 (IOVDD), U2.33 (IOVDD), U2.42 (IOVDD), U2.43 (ADC_AVDD), U2.44 (VREG_IN), U2.48 (USB_VDD), U2.49 (IOVDD), U4.5 (OUT)
- new net Col7: ENC3.S1, ENC6.S1, ENC9.S1, SW14.2, SW22.2, SW32.2, SW41.2, SW7.2, U2.40 (GPIO28_ADC2)
- new net D+: J1.A6 (D+), J1.B6 (D+), R3.2, U3.3 (IO2)
- new net D-: J1.A7 (D-), J1.B7 (D-), R4.2, U3.1 (IO1)
- new net DN: R4.1, U2.46 (USB_DM)
- new net DP: R3.1, U2.47 (USB_DP)
- new net Earth_Protective: FB2.1, FB3.1, J1.S1 (SHIELD), J2.S1 (SHIELD)
- new net Enc3: D7.2 (A), ENC3.S2, SW7.1
- new net Enc6: D30.2 (A), ENC6.S2, SW32.1
- new net Enc8: D37.2 (A), ENC8.S2, SW40.1
- new net Enc9: D38.2 (A), ENC9.S2, SW41.1
- new net EncC: C4.2, C7.1, ENC11.A, ENC4.B, ENC5.B, ENC6.B, ENC7.B, ENC8.B, ENC9.B, U2.11 (GPIO8)
- new net EncD: C5.1, C8.2, ENC10.A, ENC11.B, U2.12 (GPIO9)
- new net EncE: C6.2, ENC10.B, U2.13 (GPIO10)
- new net RX: J2.A6 (D+), J2.B6 (D+), U2.3 (GPIO1), U3.6 (IO4)
- new net TX: J2.A7 (D-), J2.B7 (D-), U2.2 (GPIO0), U3.4 (IO3)
- new net VBUS: D40.2 (A), FB1.2, R9.1, U3.5 (VP)
- new net VBUS_DETECT: R10.1, R9.2, U2.30 (GPIO19)
- no-connect marks 2 -> 16
Other:
- note added: "Power"
- moved on the sheet: C1, C3, D1, D10, D11, D12, D13, D14, D15, D16, D17, D18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
