File: v2/RefleXion 65 - PCB/RefleXion - Ortho 65.kicad_sch (KiCad schematic)
At the start: 210 parts, among them J1 USB_C_Receptacle_USB2.0, J2 USB_C_Receptacle_USB2.0, SW1 SW_Push, SW10 SW_Push, SW11 SW_Push, SW12 SW_Push, SW13 SW_Push, SW14 SW_Push, SW15 SW_Push, SW16 SW_Push, SW17 SW_Push, SW18 SW_Push, SW19 SW_Push, SW2 SW_Push, SW20 SW_Push, SW21 SW_Push, SW22 SW_Push, SW23 SW_Push, SW24 SW_Push, SW24A1 SW_Push, SW25 SW_Push, SW26 SW_Push, SW27 SW_Push, SW28 SW_Push, SW29 SW_Push, SW3 SW_Push, SW30 SW_Push, SW31 SW_Push, SW32 SW_Push, SW32A1 SW_Push, SW33 SW_Push, SW34 SW_Push, SW34A1 SW_Push, SW35 SW_Push, SW36 SW_Push, SW37 SW_Push, SW38 SW_Push, SW39 SW_Push, SW4 SW_Push, SW5 SW_Push, SW6 SW_Push, SW7 SW_Push, SW8 SW_Push, SW9 SW_Push, U1 W25Q32JVUUIQ, U2 RP2040, U3 SRV05-4, U4 SPX3819M5-L-3-3/TR, U6 SN74LV1T34DBV, Y1 TXM12M0004252LBCEO00T

Commit message: new layout
Parts:
- removed LED42: SK6812MINI-E, Keyboard RGB:MX_SK6812MINI-E_REVERSIBLE, symbol Keyboard Common:SK6812MINI-E
- added ENC12, ENC13: Rotary_Encoder_Click, Keyboard Encoders:Encoder_Alps_EC11E_Small, symbol Keyboard Switches:Rotary_Encoder_Click
- added JP10, JP13: Jumper_3_Open, Keyboard Common:SolderJumper-3_open_mini, symbol Jumper:Jumper_3_Open
- added JP14, JP15, JP16, JP17, JP18, JP19: Jumper_2_Open, Keyboard Common:Jumper_min_v2, symbol Jumper:Jumper_2_Open
- added LED34A1: SK6812MINI-E, Keyboard RGB:MX_SK6812MINI-E_REVERSIBLE_special, symbol Keyboard Common:SK6812MINI-E
- LED23, LED24, LED32: footprint Keyboard RGB:MX_SK6812MINI-E_REVERSIBLE_special -> Keyboard RGB:MX_SK6812MINI-E_REVERSIBLE
- renumbered SW24A1 to SW25A1, SW32A1 to SW33A1
Connections:
- net +5V: now also LED32A1.1 (VDD), LED44.1 (VDD), LED45.1 (VDD), LED46.1 (VDD), LED34A1.1 (VDD)
- net Col0: now also U2.15 (GPIO12), ENC12.S2, ENC13.S2; no longer SW25A1.2, SW33A1.1, U2.16 (GPIO13)
- net Col1: now also SW25.1, SW25A1.2, SW33A1.2; no longer SW25.2
- net Col2: now also SW34.2; no longer SW34.1
- net Col3: now also SW35.1; no longer SW35.2
- net Col4: now also U2.37 (GPIO25); no longer U2.35 (GPIO23)
- net Col7: now also SW39.2; no longer ENC9.S1, SW39.1
- net Enc10: now also D8.2 (A), SW8.2; no longer D16.2 (A), SW16.2
- net Enc11: now also D16.2 (A), SW16.2; no longer D8.2 (A), SW8.2
- net Enc9: now also SW39.1; no longer ENC9.S2, SW39.2
- net EncA: now also U2.35 (GPIO23); no longer U2.37 (GPIO25)
- net EncC: now also U2.16 (GPIO13), ENC13.A; no longer ENC11.A, U2.15 (GPIO12)
- net EncD: now also ENC13.B; no longer ENC11.B
- net GND: now also LED32A1.3 (GND), LED44.3 (GND), LED45.3 (GND), LED46.3 (GND), ENC12.C, ENC12.MP1 (GND), ENC12.MP2 (GND), ENC13.C, ENC13.MP1 (GND), ENC13.MP2 (GND), LED34A1.3 (GND)
- net Row2: now also U2.25 (SWD); no longer U2.14 (GPIO11)
- net Row3: now also U2.24 (SWCLK); no longer U2.13 (GPIO10)
- net at LED32A1.2 (DOUT): now also LED33.2 (DOUT), JP13.2 (C)
- net at LED32A1.4 (DIN): now also JP10.1 (A)
- net RGB_3.3: now reaches LED44.4 (DIN)
- net RGB_3.3: now also U6.4 (Y)
- net at LED29.4 (DIN), LED30.2 (DOUT): now also JP18.1 (A)
- net at LED30.4 (DIN), LED31.2 (DOUT): now also JP19.1 (A)
- net at LED22.2 (DOUT), LED23.4 (DIN): now also JP19.2 (B)
- net at LED24.2 (DOUT), LED24A1.2 (DOUT): now also JP10.2 (C); no longer LED32.4 (DIN)
- net at LED5.2 (DOUT), LED6.4 (DIN): now also JP15.2 (B)
- net at LED4.2 (DOUT), LED5.4 (DIN): now also JP16.2 (B)
- net at D24.2 (A), SW24.2: no longer SW25A1.1
- net at LED6.2 (DOUT), LED7.4 (DIN): now also JP14.2 (B)
- net at LED28.4 (DIN), LED29.2 (DOUT): now also JP17.1 (A)
- net Enc13: now reaches D32.2 (A), SW32.2
- net Enc13: now also ENC13.S1; no longer SW33A1.2
- net at D33.2 (A), SW33.1: now also SW33A1.1
- net at LED14.4 (DIN), LED15.2 (DOUT): now also JP14.1 (A)
- net at D34.2 (A), SW34A1.1: now also SW34.1; no longer SW34.2
- net at LED34.4 (DIN): now also JP13.3 (B); no longer LED33.2 (DOUT)
- net at LED20.2 (DOUT), LED21.4 (DIN): now also JP17.2 (B)
- net at LED21.2 (DOUT), LED22.4 (DIN): now also JP18.2 (B)
- net at LED13.4 (DIN), LED14.2 (DOUT): now also JP15.1 (A)
- net at LED35.2 (DOUT), LED36.4 (DIN): now also LED34A1.2 (DOUT)
- net at D25.2 (A): now also SW25.2, SW25A1.1; no longer SW25.1
- net at LED1.4 (DIN): now also LED46.2 (DOUT); no longer U6.4 (Y)
- net at LED12.4 (DIN), LED13.2 (DOUT): now also JP16.1 (A)
- net at D35.2 (A): now also SW35.2; no longer SW35.1
- new net: JP10.3 (B), LED32.4 (DIN)
- new net: JP13.1 (A), LED34A1.4 (DIN)
- new net Enc12: ENC12.S1
- no-connect marks 16 -> 15
Other:
- moved on the sheet: C7, C8, D1, D16, D17, D24, D25, D32, D33, D34, D35, D36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

Commit message: working route
Parts:
- removed FB2, FB3: BLM18SG700TZ1D, Capacitor_SMD:C_0603_1608Metric_Pad1.08x0.95mm_HandSolder, symbol LCSC Parts:Ferrite Bead
- removed JP10, JP13, JP9: Jumper_3_Open, Keyboard Common:SolderJumper-3_open_mini, symbol Jumper:Jumper_3_Open
- removed LED34A1: SK6812MINI-E, Keyboard RGB:MX_SK6812MINI-E_REVERSIBLE_special, symbol Keyboard Common:SK6812MINI-E
- removed ST3: Stabilizer_2u_MX, Keyboard Stabilizer:Stabilizer_Cherry_MX_2.00u, symbol Keyboard Switches:Stabilizer_2u_MX
- removed SW34A1: SW_Push, Keyboard Switches:SW_MX_HotSwap_Reversible, symbol Keyboard Switches:SW_MX_HotSwap_Reversible
- LED24: renamed from LED24A1; footprint Keyboard RGB:MX_SK6812MINI-E_REVERSIBLE_special -> Keyboard RGB:MX_SK6812MINI-E_REVERSIBLE
- LED25: renamed from LED24; footprint Keyboard RGB:MX_SK6812MINI-E_REVERSIBLE -> Keyboard RGB:MX_SK6812MINI-E_REVERSIBLE_special
- LED26: footprint Keyboard RGB:MX_SK6812MINI-E_REVERSIBLE -> Keyboard RGB:MX_SK6812MINI-E_REVERSIBLE_special
- LED32: renamed from LED32A1; footprint Keyboard RGB:MX_SK6812MINI-E_REVERSIBLE_special -> Keyboard RGB:MX_SK6812MINI-E_REVERSIBLE
- renumbered LED25 to LED25A1, LED32 to LED33, LED33 to LED33A1
Connections:
- net Col1: now also SW25.2, SW25A1.1; no longer SW25.1, SW25A1.2
- net Col7: now also ENC9.S1
- net Earth_Protective: no longer J1.S1 (SHIELD), J2.S1 (SHIELD)
- net Enc12: now also D24.2 (A), SW24.2
- net Enc9: now also ENC9.S2
- net EncC: now also ENC11.A, ENC12.A
- net EncD: now also ENC11.B, ENC12.B
- net GND: now also J1.S1 (SHIELD), J2.S1 (SHIELD)
- net at LED32.2 (DOUT): now also LED33.4 (DIN); no longer LED33A1.2 (DOUT)
- net at LED32.4 (DIN): now also LED24.2 (DOUT)
- net at LED25.2 (DOUT): now also LED24.4 (DIN); no longer LED24.2 (DOUT)
- net at LED26.2 (DOUT): now also LED25A1.4 (DIN)
- new net: D25.2 (A), SW25.1, SW25A1.2
Other:
- moved on the sheet: D34, LED24, LED25, LED25A1, SW34
