File: RefleXion - composite/RefleXion 65.kicad_pcb (KiCad board)
At the start: 2 copper layers, 133.4 x 117.1 mm, 152 parts, among them J1 Conn_01x21, J2 USB_C_Receptacle_USB2.0, J3 Conn_01x01, J4 Conn_01x01, J5 Conn_01x21, J6 USB_C_Receptacle_USB2.0, Q1 AO3401A, SW1 SW_Push, SW10 SW_Push, SW11 SW_Push, SW12 SW_Push, SW13 SW_Push, SW14 SW_Push, SW15 SW_Push, SW16 SW_Push, SW17 SW_Push, SW18 SW_Push, SW19 SW_Push, SW2 SW_Push, SW20 SW_Push, SW21 SW_Push, SW22 SW_Push, SW23 SW_Push, SW24 SW_Push, SW25 SW_Push, SW26 SW_Push, SW27 SW_Push, SW28 SW_Push, SW29 SW_Push, SW3 SW_Push, SW30 SW_Push, SW31 SW_Push, SW32 SW_Push, SW33 SW_Push, SW34 SW_Push, SW4 SW_Push, SW5 SW_Push, SW6 SW_Push, SW7 SW_Push, SW8 SW_Push, SW9 SW_Push, U1 WeAct_Blackpill_v3_safepin, U2 SRV05-4, U3 74AHCT1G125, U4 74AHCT1G125

Commit message: X65 initial commit
Parts:
- removed C3, C4, C5, C6: 100nF, Capacitor_SMD:C_0603_1608Metric_Pad1.08x0.95mm_HandSolder
- removed the ENC1 at (53.7, 47.5)
- removed ENC2: Rotary_Encoder_Click, Keyboard Encoders:Encoder_Alps_EC11E_Small
- removed FB1, FB2: FerriteBead_Small, Capacitor_SMD:C_0805_2012Metric_Pad1.18x1.45mm_HandSolder
- removed H5, H6: Spacer_Plate, Keyboard_Plate:Spacer Plate hole
- removed J1, J5: Conn_01x21, Connector_PinHeader_2.54mm:PinHeader_1x21_P2.54mm_Vertical
- removed J2, J6: USB_C_Receptacle_USB2.0, Keyboard Common:HRO_TYPE-C-31-M-12
- removed J3, J4: Conn_01x01, Connector_PinHeader_2.54mm:PinHeader_1x01_P2.54mm_Vertical
- removed JP1, JP2, JP3, JP4, JP5, JP6, JP7, JP8: Jumper_NO_Small, Keyboard Common:Jumper_Mini
- removed Logo1: CC-BY-SA-4.0, Logotypes:CC_BY_SA_40
- removed Logo2: QMK_Logo, Logotypes:Powered_by_QMK
- removed Q1: AO3401A, Package_TO_SOT_SMD:SOT-23
- removed R1, R2, R3, R4, R5, R6: 9.1k, Resistor_SMD:R_0603_1608Metric_Pad0.98x0.95mm_HandSolder
- removed U3, U4: 74AHCT1G125, Package_TO_SOT_SMD:SOT-353_SC-70-5_Handsoldering
- added BOOT1: YTS-A002, Keyboard Common:YTS-A002, B.Cu at (116.0, 17.5)
- added C10: 100nF, Capacitor_SMD:C_0402_1005Metric, B.Cu at (122.1, 36.5)
- added C11: 100nF, Capacitor_SMD:C_0402_1005Metric, B.Cu at (122.1, 37.5)
- added C12: 100nF, Capacitor_SMD:C_0402_1005Metric, B.Cu at (124.2, 27.8)
- added C13: 1uF, Capacitor_SMD:C_0402_1005Metric, B.Cu at (133.0, 34.8)
- added C14: 100nF, Capacitor_SMD:C_0402_1005Metric, B.Cu at (120.4, 30.8)
- added C15: 100nF, Capacitor_SMD:C_0402_1005Metric, B.Cu at (122.1, 35.6)
- added C16: 1uF, Capacitor_SMD:C_0402_1005Metric, B.Cu at (96.1, 30.1)
- added C17: 1uF, Capacitor_SMD:C_0402_1005Metric, B.Cu at (128.0, 38.0)
- added C18: 100nF, Capacitor_SMD:C_0402_1005Metric, B.Cu at (120.4, 32.6)
- added C19: 30pF, Capacitor_SMD:C_0402_1005Metric, B.Cu at (137.9, 32.9)
- added C20: 30pF, Capacitor_SMD:C_0402_1005Metric, B.Cu at (134.9, 30.3)
- added C7: 1uF, Capacitor_SMD:C_0402_1005Metric, B.Cu at (128.2, 27.6)
- added C8: 100nF, Capacitor_SMD:C_0402_1005Metric, B.Cu at (133.0, 33.8)
- added C9: 100nF, Capacitor_SMD:C_0402_1005Metric, B.Cu at (120.4, 31.7)
- added F1: CF06V5TR50, Resistor_SMD:R_0603_1608Metric, B.Cu at (96.2, 27.0)
- added FB3: BLM18SG700TZ1D, Capacitor_SMD:C_0603_1608Metric_Pad1.08x0.95mm_HandSolder, B.Cu at (143.8, 24.5)
- added FB4: BLM18SG700TZ1D, Capacitor_SMD:C_0603_1608Metric_Pad1.08x0.95mm_HandSolder, B.Cu at (77.5, 21.9)
- added JP10: Jumper_2_Open, Keyboard Common:Jumper_min_v2, F.Cu at (106.5, 24.3)
- added JP11: Jumper_2_Open, Keyboard Common:Jumper_min_v2, F.Cu at (106.5, 26.8)
- added JP12: Jumper_2_Open, Keyboard Common:Jumper_min_v2, F.Cu at (106.5, 29.4)
- added JP13: Jumper_2_Open, Keyboard Common:Jumper_min_v2, B.Cu at (106.5, 21.7)
- added JP14: Jumper_2_Open, Keyboard Common:Jumper_min_v2, B.Cu at (106.5, 24.3)
- added JP15: Jumper_2_Open, Keyboard Common:Jumper_min_v2, B.Cu at (106.5, 26.8)
- added JP16: Jumper_2_Open, Keyboard Common:Jumper_min_v2, B.Cu at (106.5, 29.4)
- added JP17: Jumper_3_Open, Keyboard Common:SolderJumper-3_open_mini, B.Cu at (141.8, 37.6)
- added JP9: Jumper_2_Open, Keyboard Common:Jumper_min_v2, F.Cu at (106.5, 21.7)
- added Logo3: CC-BY-SA-4.0, Logotypes:CC_BY_SA_40_line, F.Cu at (92.0, 36.9)
- added Logo4: QMK_Logo, Logotypes:Powered_by_QMK, F.Cu at (126.4, 37.0)
- added R10: 68K, Resistor_SMD:R_0402_1005Metric, B.Cu at (129.4, 38.0)
- added R11: 68K, Resistor_SMD:R_0402_1005Metric, B.Cu at (129.8, 39.4)
- added R12: 10K, Resistor_SMD:R_0402_1005Metric, B.Cu at (131.7, 37.6)
- added R13: 10K, Resistor_SMD:R_0402_1005Metric, B.Cu at (117.8, 28.2)
- added R14: 1K, Resistor_SMD:R_0402_1005Metric, B.Cu at (117.8, 26.2)
- added R15: 1K, Resistor_SMD:R_0402_1005Metric, B.Cu at (133.4, 32.4)
- added R16: 27R, Resistor_SMD:R_0402_1005Metric, B.Cu at (116.5, 33.7)
- added R17: 27R, Resistor_SMD:R_0402_1005Metric, B.Cu at (116.5, 34.6)
- added R18: 10K, Resistor_SMD:R_0402_1005Metric, B.Cu at (133.0, 35.7)
- added R7: 5.1K, Resistor_SMD:R_0402_1005Metric, B.Cu at (76.9, 29.4)
- added R8: 5.1K, Resistor_SMD:R_0402_1005Metric, B.Cu at (77.0, 24.5)
- added R9: 68K, Resistor_SMD:R_0402_1005Metric, B.Cu at (130.3, 38.0)
- added RES1: YTS-A002, Keyboard Common:YTS-A002, B.Cu at (128.6, 17.5)
- added SW35: SW_Push, Keyboard Switches:SW_MX_HotSwap_Reversible, F.Cu at (158.5, 123.7)
- added SW36: SW_Push, Keyboard Switches:SW_MX_HotSwap_Reversible, F.Cu at (168.0, 123.7)
- added U5: SPX3819M5-L-3-3/TR, Package_TO_SOT_SMD:SOT-23-5, B.Cu at (99.0, 29.6)
- added U6: SRV05-4, Package_TO_SOT_SMD:SOT-23-6, B.Cu at (93.0, 33.6)
- added U7: W25Q32JVUUIQ, Keyboard Common:USON-8_4x3mm_P0.8mm, B.Cu at (120.6, 27.2)
- added U8: RP2040, Package_DFN_QFN:QFN-56-1EP_7x7mm_P0.4mm_EP3.2x3.2mm, B.Cu at (127.2, 32.9)
- added USB1: USB_C_Receptacle_USB2.0, Keyboard Common:Molex-216990_GCT-USB45xx_HRO-TYPE-C-31-M-13x-PiMicro, B.Cu at (68.5, 26.9)
- added USB2: USB_C_Receptacle_USB2.0, Keyboard Common:Molex-216990_GCT-USB45xx_HRO-TYPE-C-31-M-13x-PiMicro, B.Cu at (153.3, 26.9)
- added Y1: TXM12M0004252LBCEO00T, Crystal:Crystal_SMD_2520-4Pin_2.5x2.0mm, B.Cu at (135.7, 32.3)
- added ZD1: 1N5819WS, Diode_SMD:D_SOD-323F, B.Cu at (96.3, 25.1)
- C1, C2: footprint Capacitor_SMD:C_0603_1608Metric_Pad1.08x0.95mm_HandSolder -> Capacitor_SMD:C_0402_1005Metric
- D36: value SMF5.0CA -> 1N4148W; footprint Diode_SMD:D_SOD-123F -> Diode_SMD:D_SOD-123; moved to B.Cu
- LED34, LED35, LED36: footprint Keyboard RGB:MX_SK6812MINI-E_REVERSIBLE -> Keyboard RGB:MX_SK6812MINI-E_REVERSIBLE_special
- U1: value WeAct_Blackpill_v3_safepin -> SN74LV1T34DBV; footprint Keyboard Controllers:WeAct_BlackPill_3_reverse_mount -> Package_TO_SOT_SMD:SOT-23-5; moved to B.Cu
- U2: moved to B.Cu
- moved D35 118.5 mm to (163.0, 114.5)
- moved D36 114.8 mm to (83.9, 36.1), turned to 180 degrees
- moved LED35 111.9 mm to (158.5, 118.6), turned to -90 degrees
- moved LED36 111.7 mm to (168.0, 128.7), turned to 90 degrees
- moved U2 111.5 mm to (137.2, 26.4)
- moved C2 99.6 mm to (78.2, 18.0)
- moved C1 86.2 mm to (89.7, 18.0)
- moved U1 71.2 mm to (114.7, 37.6), turned to 180 degrees
- moved D8 17.2 mm to (61.8, 68.5)
- moved D1 17.0 mm to (61.9, 49.7)
- moved D29 16.7 mm to (61.8, 125.7), turned to 90 degrees
- moved D15 16.6 mm to (61.8, 87.6), turned to 90 degrees
- moved D22 16.5 mm to (61.8, 106.6), turned to 90 degrees
- moved D34 12.1 mm to (154.0, 114.5), turned to 180 degrees
- moved LED34 9.52 mm to (149.0, 128.7), turned to 90 degrees
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- renumbered ENC3 to ENC1
Connections:
- C1 pad 1: B1 -> EncA
- C2 pad 2: A2 -> EncB
- D1 pad 1: Row0 -> Row1
- D10 pad 1: Row1 -> Row2
- D11 pad 1: Row1 -> Row2
- D12 pad 1: Row1 -> Row2
- D13 pad 1: Row1 -> Row2
- D14 pad 1: Row1 -> Row2
- D15 pad 1: Row2 -> Row3
- D15 pad 2: Net-(D15-Pad2) -> Net-(D15-A)
- D16 pad 1: Row2 -> Row3
- D17 pad 1: Row2 -> Row3
- D18 pad 1: Row2 -> Row3
- D19 pad 1: Row2 -> Row3
- D2 pad 1: Row0 -> Row1
- D20 pad 1: Row2 -> Row3
- D21 pad 1: Row2 -> Row3
- D22 pad 1: Row3 -> Row4
- D22 pad 2: Net-(D22-Pad2) -> Net-(D22-A)
- D23 pad 1: Row3 -> Row4
- D24 pad 1: Row3 -> Row4
- D25 pad 1: Row3 -> Row4
- D26 pad 1: Row3 -> Row4
- D27 pad 1: Row3 -> Row4
- D28 pad 1: Row3 -> Row4
- D29 pad 1: Row4 -> Row5
- D29 pad 2: Net-(D29-Pad2) -> Net-(D29-A)
- D3 pad 1: Row0 -> Row1
- D30 pad 1: Row4 -> Row5
- D31 pad 1: Row4 -> Row5
- D32 pad 1: Row4 -> Row5
- D33 pad 1: Row4 -> Row5
- D34 pad 1: Row4 -> Row5
- D35 pad 1: Row4 -> Row5
- D35 pad 2: Net-(D35-Pad2) -> Net-(D35-A)
- D36 pad 1: GND -> Row0
- D36 pad 2: Net-(D36-Pad2) -> Net-(D36-A)
- D4 pad 1: Row0 -> Row1
- D5 pad 1: Row0 -> Row1
- D6 pad 1: Row0 -> Row1
- D7 pad 1: Row0 -> Row1
- D8 pad 1: Row1 -> Row2
- D8 pad 2: Net-(D8-Pad2) -> Net-(D8-A)
- D9 pad 1: Row1 -> Row2
- ENC1 pad A: A2 -> EncA
- ENC1 pad B: B2 -> EncB
- ENC1 pad S1: Col6 -> Col1
- ENC1 pad S2: Net-(D35-Pad2) -> Net-(D36-A)
- LED1 pad 1: VCC -> +5V
- LED1 pad 4: Net-(LED1-Pad4) -> Net-(LED1-DIN)
- LED10 pad 1: VCC -> +5V
- LED11 pad 1: VCC -> +5V
- LED12 pad 1: VCC -> +5V
- LED13 pad 1: VCC -> +5V
- LED14 pad 1: VCC -> +5V
- LED15 pad 1: VCC -> +5V
- LED16 pad 1: VCC -> +5V
- LED17 pad 1: VCC -> +5V
- LED18 pad 1: VCC -> +5V
- LED19 pad 1: VCC -> +5V
- LED2 pad 1: VCC -> +5V
- LED20 pad 1: VCC -> +5V
- LED21 pad 1: VCC -> +5V
- LED22 pad 1: VCC -> +5V
- LED23 pad 1: VCC -> +5V
- LED24 pad 1: VCC -> +5V
- LED25 pad 1: VCC -> +5V
- LED26 pad 1: VCC -> +5V
- LED27 pad 1: VCC -> +5V
- LED28 pad 1: VCC -> +5V
- LED29 pad 1: VCC -> +5V
- LED3 pad 1: VCC -> +5V
- LED30 pad 1: VCC -> +5V
- LED31 pad 1: VCC -> +5V
- LED32 pad 1: VCC -> +5V
- LED33 pad 1: VCC -> +5V
- LED34 pad 1: VCC -> +5V
- LED34 pad 2: unconnected-(LED34-Pad2) -> Net-(LED34-DOUT)
- LED35 pad 1: VCC -> +5V
- LED35 pad 4: Net-(LED35-Pad4) -> Net-(LED34-DOUT)
- LED36 pad 1: VCC -> +5V
- LED4 pad 1: VCC -> +5V
- LED5 pad 1: VCC -> +5V
- LED6 pad 1: VCC -> +5V
- LED7 pad 1: VCC -> +5V
- LED8 pad 1: VCC -> +5V
- LED9 pad 1: VCC -> +5V
- SW1 pad 1: Enc1 -> Col0
- SW1 pad 2: Col0 -> Enc1
- SW15 pad 1: Net-(D15-Pad2) -> Col0
- SW15 pad 2: Col0 -> Net-(D15-A)
- SW22 pad 1: Net-(D22-Pad2) -> Col0
- SW22 pad 2: Col0 -> Net-(D22-A)
- SW29 pad 1: Net-(D29-Pad2) -> Col0
- SW29 pad 2: Col0 -> Net-(D29-A)
- SW8 pad 1: Net-(D8-Pad2) -> Col0
- SW8 pad 2: Col0 -> Net-(D8-A)
- U1 pad 1: Col0 -> unconnected-(U1-NC-Pad1)
- U1 pad 2: Col1 -> RGB
- U1 pad 3: A1 -> GND
- U1 pad 4: B1 -> Net-(LED1-DIN)
- U1 pad 5: Row0 -> +5V
- U2 pad 1: TX -> SER-
- U2 pad 3: RX -> SER+
- U2 pad 4: unconnected-(U2-Pad4) -> SER+
- U2 pad 5: VCC -> +5V
- U2 pad 6: unconnected-(U2-Pad6) -> SER-
Routing:
- net VCC: track 996.2 -> 0.00 mm, vias 57 -> 0
- net +5V: track 0.00 -> 876.5 mm, vias 0 -> 47
- net Row5: track 0.00 -> 210.9 mm, vias 0 -> 2
- net Col1: track 0.00 -> 157.5 mm, vias 0 -> 13
- net B1: track 134.5 -> 0.00 mm, vias 1 -> 0
- net A2: track 115.6 -> 0.00 mm, vias 2 -> 0
- net Net-(LED1-DIN): track 0.00 -> 99.5 mm, vias 0 -> 5
- net Row0: track 163.4 -> 78.0 mm, vias 8 -> 2
- net +3V3: track 0.00 -> 81.9 mm, vias 0 -> 6
- net VBUS: track 0.00 -> 76.1 mm, vias 0 -> 5
- net Col0: track 104.3 -> 178.4 mm, vias 10 -> 13
- net Row4: track 236.2 -> 175.2 mm, vias 7 -> 2
- net EncB: track 0.00 -> 57.8 mm, vias 0 -> 2
- net Row1: track 173.9 -> 117.1 mm, vias 9 -> 2
- net A1: track 55.6 -> 0.00 mm, vias 1 -> 0
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Other:
- outline, holes or cut-outs redrawn
- board text added: "Close for OLED on LEFT Hand"
- board text added: "Close for OLED on RIGHT Hand"
- board text added: "LH"
- board text added: "RH"
- board text added: "RefleXion X65 - v1.10 - 2024"
- board text added: "Set Hand"
- board text added: "TO HOST"
- board text added: "USB Link"
- board text removed: "Large RGB Module - 2022 Design: Markus Knutsson - Concept: Pedro Quaresma https://github.com/TweetyDaBird"
- board text removed: "RefleXion - Ortho 65 Matrix - 2022"
