File: RefleXion - composite/RefleXion 65.kicad_sch (KiCad schematic)
At the start: 121 parts, among them J1 Conn_01x25, SW1 SW_Push, SW10 SW_Push, SW11 SW_Push, SW12 SW_Push, SW13 SW_Push, SW14 SW_Push, SW15 SW_Push, SW16 SW_Push, SW17 SW_Push, SW18 SW_Push, SW19 SW_Push, SW2 SW_Push, SW20 SW_Push, SW21 SW_Push, SW22 SW_Push, SW23 SW_Push, SW24 SW_Push, SW25 SW_Push, SW26 SW_Push, SW27 SW_Push, SW28 SW_Push, SW29 SW_Push, SW3 SW_Push, SW30 SW_Push, SW31 SW_Push, SW32 SW_Push, SW33 SW_Push, SW34 SW_Push, SW4 SW_Push, SW5 SW_Push, SW6 SW_Push, SW7 SW_Push, SW8 SW_Push, SW9 SW_Push

Commit message: Adding Reflexion 60
Parts:
- added D36: SMF5.0CA, Diode_SMD:D_SOD-123F, symbol Keyboard Common:SMF5.0CA
- added FB1, FB2: FerriteBead_Small, Capacitor_SMD:C_0805_2012Metric_Pad1.18x1.45mm_HandSolder, symbol Device:FerriteBead_Small
- added J2, J6: USB_C_Receptacle_USB2.0, Keyboard Common:HRO_TYPE-C-31-M-12, symbol Connector:USB_C_Receptacle_USB2.0
- added J3, J4: Conn_01x01, Connector_PinHeader_2.54mm:PinHeader_1x01_P2.54mm_Vertical, symbol Connector_Generic:Conn_01x01
- added J5: Conn_01x21, Connector_PinHeader_2.54mm:PinHeader_1x21_P2.54mm_Vertical, symbol Connector_Generic:Conn_01x21
- added JP1, JP2, JP3, JP4, JP5, JP6, JP7, JP8: Jumper_NO_Small, Keyboard Common:Jumper_Mini, symbol Device:Jumper_NO_Small
- added LED35, LED36: SK6812MINI-E, Keyboard RGB:MX_SK6812MINI-E_REVERSIBLE, symbol Keyboard Common:SK6812MINI-E
- added Logo1: CC-BY-SA-4.0, Logotypes:CC_BY_SA_40, symbol Logotypes:CC-BY-SA-4.0
- added Logo2: QMK_Logo, Logotypes:Powered_by_QMK, symbol Logotypes:QMK_Logo
- added Q1: AO3401A, Package_TO_SOT_SMD:SOT-23, symbol Transistor_FET:AO3401A
- added R1, R2, R3, R4, R5, R6: 9.1k, Resistor_SMD:R_0603_1608Metric_Pad0.98x0.95mm_HandSolder, symbol Device:R_Small
- added U1: WeAct_Blackpill_v3_safepin, Keyboard Controllers:WeAct_BlackPill_3_reverse_mount, symbol Keyboard Controllers:WeAct_Blackpill_v3_safepin
- added U2: SRV05-4, Package_TO_SOT_SMD:SOT-23-6, symbol Power_Protection:SRV05-4
- added U3, U4: 74AHCT1G125, Package_TO_SOT_SMD:SOT-353_SC-70-5_Handsoldering, symbol 74xGxx:74AHCT1G125
- J1: value Conn_01x25 -> Conn_01x21; footprint Connector_PinHeader_2.54mm:PinHeader_1x25_P2.54mm_Vertical -> Connector_PinHeader_2.54mm:PinHeader_1x21_P2.54mm_Vertical; symbol Connector_Generic:Conn_01x25 -> Connector_Generic:Conn_01x21
- renumbered ENC2 to ENC1, ENC1 to ENC2
Connections:
- net A1: now also J5.6 (Pin_6), U1.3 (PB14)
- net A2: now also C2.2, C5.1, ENC2.B, ENC3.A, J1.9 (Pin_9), J5.9 (Pin_9), U1.16 (PB8); no longer C1.1, ENC2.A, J1.19 (Pin_19)
- net B1: now also C1.1, ENC2.A, J5.7 (Pin_7), U1.4 (PB15)
- net B2: now also C6.2, ENC3.B, J1.10 (Pin_10), J5.10 (Pin_10), U1.17 (PB9); no longer C2.2, ENC2.B, J1.20 (Pin_20)
- net Col0: now also J1.3 (Pin_3), J5.3 (Pin_3), U1.1 (PB12); no longer J1.4 (Pin_4)
- net Col1: now also J5.5 (Pin_5), U1.2 (PB13)
- net Col2: now also J5.11 (Pin_11), U1.34 (PB0)
- net Col3: now also J5.18 (Pin_18), U1.33 (PA7)
- net Col4: now also J1.19 (Pin_19), J5.19 (Pin_19), U1.32 (PA6); no longer J1.21 (Pin_21)
- net Col5: now also J1.20 (Pin_20), J5.20 (Pin_20), U1.31 (PA5); no longer J1.22 (Pin_22)
- net Col6: now also J1.21 (Pin_21), J5.21 (Pin_21), U1.30 (PA4); no longer J1.23 (Pin_23)
- net GND: now also D36.1 (A1), FB2.2, J2.A1 (GND), J2.A12 (GND), J2.B1 (GND), J2.B12 (GND), J5.1 (Pin_1), J6.A1 (GND), J6.A12 (GND), J6.B1 (GND), J6.B12 (GND), JP1.2, JP8.2, LED35.3 (GND), LED36.3 (GND), Q1.1 (G), R2.2, U1.19 (GND), U1.39 (GND), U2.2 (VN), U3.3 (GND), U4.3 (GND); no longer J1.25 (Pin_25), OLED1.1 (GND)
- net RGB: now also J1.4 (Pin_4), J5.4 (Pin_4), U1.35 (PB1), U3.2, U4.2; no longer J1.3 (Pin_3), LED1.4 (DIN)
- net Row0: now also J5.8 (Pin_8), U1.5 (PA8)
- net Row1: now also J5.15 (Pin_15), U1.13 (PB5)
- net Row2: now also J5.14 (Pin_14), U1.12 (PB4)
- net Row3: now also J5.13 (Pin_13), U1.11 (PB3)
- net Row4: now also J5.12 (Pin_12), U1.10 (PA15)
- net SCL: now also J5.16 (Pin_16), JP3.2, JP6.2, U1.14 (PB6); no longer OLED1.3 (SCL)
- net SDA: now also J5.17 (Pin_17), JP4.2, JP5.2, U1.15 (PB7); no longer OLED1.4 (SDA)
- net VCC: now also J5.2 (Pin_2), JP2.2, JP7.2, LED35.1 (VDD), LED36.1 (VDD), Q1.2 (S), U1.18 (5V), U1.40 (5V), U2.5 (VP), U3.1, U3.5 (VCC), U4.1, U4.5 (VCC); no longer J1.24 (Pin_24), OLED1.2 (VCC)
- removed net A3: C5.1, ENC3.A, J1.10 (Pin_10)
- removed net B3: C6.2, ENC3.B, J1.9 (Pin_9)
- net Enc3: no longer names the net of D35.2 (A), ENC3.S2
- new net: JP1.1, JP5.1, OLED1.1 (GND)
- new net: JP2.1, JP6.1, OLED1.2 (VCC)
- new net: JP3.1, JP7.1, OLED1.3 (SCL)
- new net: JP4.1, JP8.1, OLED1.4 (SDA)
- new net: LED35.2 (DOUT), LED36.4 (DIN)
- new net: LED35.4 (DIN), U4.4
- new net: LED1.4 (DIN), U3.4
- new net: FB2.1, J2.S1 (SHIELD), J6.S1 (SHIELD)
- new net: FB1.1, J2.A4 (VBUS), J2.A9 (VBUS), J2.B4 (VBUS), J2.B9 (VBUS), J6.A4 (VBUS), J6.A9 (VBUS), J6.B4 (VBUS), J6.B9 (VBUS)
- new net: J2.A5 (CC1), J6.A5 (CC1)
- new net: J2.A6 (D+), J6.A6 (D+)
- new net: J2.A7 (D-), J6.A7 (D-)
- new net: J2.B5 (CC2), J6.B5 (CC2)
- new net: J2.B6 (D+), J6.B6 (D+)
- new net: J2.B7 (D-), J6.B7 (D-)
- new net: D36.2 (A2), FB1.2, Q1.3 (D)
- new net +3.3V: R1.1, R3.1, R4.1, R5.1, R6.1, U1.20 (3V3), U1.38 (3V3)
- new net Hand: R1.2, R2.1, U1.23 (PC14)
- new net RX: J2.A8 (SBU1), J6.A8 (SBU1), R4.2, R6.2, U1.29 (PA3), U2.3 (IO2)
- new net TX: J2.B8 (SBU2), J6.B8 (SBU2), R3.2, R5.2, U1.28 (PA2), U2.1 (IO1)
- no-connect marks 1 -> 13
Other:
- moved on the sheet: C1, C2, C5, C6, D35, ENC2, ENC3, OLED1

Commit message: X65 initial commit
Parts:
- removed C3, C4, C5, C6: 100nF, Capacitor_SMD:C_0603_1608Metric_Pad1.08x0.95mm_HandSolder, symbol Device:C_Small
- removed D36: SMF5.0CA, Diode_SMD:D_SOD-123F, symbol Keyboard Common:SMF5.0CA
- removed ENC2, ENC3: Rotary_Encoder_Click, Keyboard Encoders:Encoder_Alps_EC11E_Small, symbol Keyboard Switches:Rotary_Encoder_Click
- removed FB1, FB2: FerriteBead_Small, Capacitor_SMD:C_0805_2012Metric_Pad1.18x1.45mm_HandSolder, symbol Device:FerriteBead_Small
- removed H5, H6: Spacer_Plate, Keyboard_Plate:Spacer Plate hole, symbol Keyboard_Plate:Spacer_Plate
- removed J1, J5: Conn_01x21, Connector_PinHeader_2.54mm:PinHeader_1x21_P2.54mm_Vertical, symbol Connector_Generic:Conn_01x21
- removed J2, J6: USB_C_Receptacle_USB2.0, Keyboard Common:HRO_TYPE-C-31-M-12, symbol Connector:USB_C_Receptacle_USB2.0
- removed J3, J4: Conn_01x01, Connector_PinHeader_2.54mm:PinHeader_1x01_P2.54mm_Vertical, symbol Connector_Generic:Conn_01x01
- removed JP1, JP2, JP3, JP4, JP5, JP6, JP7, JP8: Jumper_NO_Small, Keyboard Common:Jumper_Mini, symbol Device:Jumper_NO_Small
- removed Logo1: CC-BY-SA-4.0, Logotypes:CC_BY_SA_40, symbol Logotypes:CC-BY-SA-4.0
- removed Logo2: QMK_Logo, Logotypes:Powered_by_QMK, symbol Logotypes:QMK_Logo
- removed Q1: AO3401A, Package_TO_SOT_SMD:SOT-23, symbol Transistor_FET:AO3401A
- removed R1, R2, R3, R4, R5, R6: 9.1k, Resistor_SMD:R_0603_1608Metric_Pad0.98x0.95mm_HandSolder, symbol Device:R_Small
- removed U1: WeAct_Blackpill_v3_safepin, Keyboard Controllers:WeAct_BlackPill_3_reverse_mount, symbol Keyboard Controllers:WeAct_Blackpill_v3_safepin
- removed U2: SRV05-4, Package_TO_SOT_SMD:SOT-23-6, symbol Power_Protection:SRV05-4
- removed U3, U4: 74AHCT1G125, Package_TO_SOT_SMD:SOT-353_SC-70-5_Handsoldering, symbol 74xGxx:74AHCT1G125
- added BOOT1, RES1: YTS-A002, Keyboard Common:YTS-A002, symbol Keyboard Common:TS-A002
- added C10, C11, C12, C14, C15, C18, C8, C9: 100nF, Capacitor_SMD:C_0402_1005Metric, symbol Device:C
- added C13, C16, C17, C7: 1uF, Capacitor_SMD:C_0402_1005Metric, symbol Device:C
- added C19, C20: 30pF, Capacitor_SMD:C_0402_1005Metric, symbol Device:C
- added D36: 1N4148W, Diode_SMD:D_SOD-123, symbol Diode:1N4148W
- added F1: CF06V5TR50, Resistor_SMD:R_0603_1608Metric, symbol Device:Polyfuse_Small
- added FB3, FB4: BLM18SG700TZ1D, Capacitor_SMD:C_0603_1608Metric_Pad1.08x0.95mm_HandSolder, symbol LCSC Parts:Ferrite Bead
- added JP10, JP11, JP12, JP13, JP14, JP15, JP16, JP9: Jumper_2_Open, Keyboard Common:Jumper_min_v2, symbol Jumper:Jumper_2_Open
- added JP17: Jumper_3_Open, Keyboard Common:SolderJumper-3_open_mini, symbol Jumper:Jumper_3_Open
- added Logo3: CC-BY-SA-4.0, Logotypes:CC_BY_SA_40_line, symbol Logotypes:CC-BY-SA-4.0
- added Logo4: QMK_Logo, Logotypes:Powered_by_QMK, symbol Logotypes:QMK_Logo
- added R10, R11, R9: 68K, Resistor_SMD:R_0402_1005Metric, symbol Device:R_Small
- added R12, R13, R18: 10K, Resistor_SMD:R_0402_1005Metric, symbol Device:R
- added R14, R15: 1K, Resistor_SMD:R_0402_1005Metric, symbol Device:R
- added R16, R17: 27R, Resistor_SMD:R_0402_1005Metric, symbol Device:R_Small
- added R7, R8: 5.1K, Resistor_SMD:R_0402_1005Metric, symbol Device:R_Small
- added SW35, SW36: SW_Push, Keyboard Switches:SW_MX_HotSwap_Reversible, symbol Keyboard Switches:SW_MX_HotSwap_Reversible
- added U1: SN74LV1T34DBV, Package_TO_SOT_SMD:SOT-23-5, symbol Logic_LevelTranslator:SN74LV1T34DBV
- added U2, U6: SRV05-4, Package_TO_SOT_SMD:SOT-23-6, symbol LCSC Parts:SRV05-4
- added U5: SPX3819M5-L-3-3/TR, Package_TO_SOT_SMD:SOT-23-5, symbol Regulator_Linear:SPX3819M5-L-3-3
- added U7: W25Q32JVUUIQ, Keyboard Common:USON-8_4x3mm_P0.8mm, symbol Memory_Flash:W25Q32JVSS
- added U8: RP2040, Package_DFN_QFN:QFN-56-1EP_7x7mm_P0.4mm_EP3.2x3.2mm, symbol MCU_RaspberryPi:RP2040
- added USB1: USB_C_Receptacle_USB2.0, Keyboard Common:Molex-216990_GCT-USB45xx_HRO-TYPE-C-31-M-13x-PiMicro, symbol Connector:USB_C_Receptacle_USB2.0
- added USB2: USB_C_Receptacle_USB2.0, Keyboard Common:Molex-216990_GCT-USB45xx_HRO-TYPE-C-31-M-13x-PiMicro, symbol Connector:USB_C_Receptacle_USB2.0_16P
- added Y1: TXM12M0004252LBCEO00T, Crystal:Crystal_SMD_2520-4Pin_2.5x2.0mm, symbol Device:Crystal_GND24
- added ZD1: 1N5819WS, Diode_SMD:D_SOD-323F, symbol Device:D_Schottky_Small
- C1, C2: footprint Capacitor_SMD:C_0603_1608Metric_Pad1.08x0.95mm_HandSolder -> Capacitor_SMD:C_0402_1005Metric; LCSC (none) -> C513772
- D1, D10, D11, D12, D13, D14, D15, D16, D17, D18, D19, D2, D20, D21, D22, D23, D24, D25, D26, D27, D28, D29, D3, D30, D31, D32, D33, D34, D35, D4, D5, D6, D7, D8, D9: LCSC (none) -> C81598
- LED34, LED35, LED36: footprint Keyboard RGB:MX_SK6812MINI-E_REVERSIBLE -> Keyboard RGB:MX_SK6812MINI-E_REVERSIBLE_special
- ST1: now not fitted
Connections:
- net Col0: now also SW1.1, SW15.1, SW22.1, SW29.1, SW8.1, U8.39 (GPIO27_ADC1); no longer ENC1.S1, SW1.2, SW15.2, SW22.2, SW29.2, SW8.2
- net Col1: now also ENC1.S1, U8.38 (GPIO26_ADC0)
- net Col2: now also U8.37 (GPIO25)
- net Col3: now also U8.41 (GPIO29_ADC3)
- net Col4: now also U8.15 (GPIO12)
- net Col5: now also U8.14 (GPIO11)
- net Col6: now also SW35.1, SW36.2, U8.13 (GPIO10)
- net Enc1: now also SW1.2; no longer ENC1.S2, SW1.1
- net GND: now also BOOT1.2, BOOT1.3, C10.2, C11.2, C12.2, C13.2, C14.2, C15.2, C16.2, C17.2, C18.2, C19.2, C20.2, C7.2, C8.2, C9.2, JP12.1 (A), JP13.1 (A), JP17.1 (A), R11.2, R7.1, R8.2, RES1.2, RES1.3, U1.3 (GND), U2.2 (VN), U5.2 (GND), U6.2 (VN), U7.4 (GND), U8.19 (TESTEN), U8.57 (GND), USB1.A1 (GND), USB1.A12 (GND), USB1.B1 (GND), USB1.B12 (GND), USB1.S1 (SHIELD), USB2.A1 (GND), USB2.A12 (GND), USB2.B1 (GND), USB2.B12 (GND), USB2.S1 (SHIELD), Y1.2, Y1.4
- net RGB: now also U1.2 (A), U8.31 (GPIO20)
- net Row0: now also D36.1 (K), U8.16 (GPIO13); no longer D1.1 (K), D2.1 (K), D3.1 (K), D4.1 (K), D5.1 (K), D6.1 (K), D7.1 (K)
- net Row1: now also D1.1 (K), D2.1 (K), D3.1 (K), D4.1 (K), D5.1 (K), D6.1 (K), D7.1 (K), U8.40 (GPIO28_ADC2); no longer D10.1 (K), D11.1 (K), D12.1 (K), D13.1 (K), D14.1 (K), D8.1 (K), D9.1 (K)
- net Row2: now also D10.1 (K), D11.1 (K), D12.1 (K), D13.1 (K), D14.1 (K), D8.1 (K), D9.1 (K), U8.36 (GPIO24); no longer D15.1 (K), D16.1 (K), D17.1 (K), D18.1 (K), D19.1 (K), D20.1 (K), D21.1 (K)
- net Row3: now also D15.1 (K), D16.1 (K), D17.1 (K), D18.1 (K), D19.1 (K), D20.1 (K), D21.1 (K), U8.35 (GPIO23); no longer D22.1 (K), D23.1 (K), D24.1 (K), D25.1 (K), D26.1 (K), D27.1 (K), D28.1 (K)
- net Row4: now also D22.1 (K), D23.1 (K), D24.1 (K), D25.1 (K), D26.1 (K), D27.1 (K), D28.1 (K), U8.34 (GPIO22); no longer D29.1 (K), D30.1 (K), D31.1 (K), D32.1 (K), D33.1 (K), D34.1 (K), D35.1 (K)
- net SCL: now also JP10.1 (A), JP15.1 (A), U8.28 (GPIO17)
- net SDA: now also JP16.1 (A), JP9.1 (A), U8.27 (GPIO16)
- net at OLED1.1 (GND): now also JP12.2 (B), JP16.2 (B)
- net at OLED1.2 (VCC): now also JP11.2 (B), JP15.2 (B)
- net at OLED1.3 (SCL): now also JP10.2 (B), JP14.2 (B)
- net at OLED1.4 (SDA): now also JP13.2 (B), JP9.2 (B)
- net at D29.2 (A): now also SW29.2; no longer SW29.1
- net at D35.2 (A): now also SW35.2, SW36.1
- net at LED34.2 (DOUT): now also LED35.4 (DIN)
- net at D15.2 (A): now also SW15.2; no longer SW15.1
- net at D22.2 (A): now also SW22.2; no longer SW22.1
- net at D8.2 (A): now also SW8.2; no longer SW8.1
- net at LED1.4 (DIN): now also U1.4 (Y)
- net A1 renamed EncA
- net EncA: now also C1.1, U8.8 (GPIO6)
- net A2 renamed EncB
- net EncB: now also ENC1.B, U8.7 (GPIO5)
- removed net B1: C1.1, ENC1.B
- net VCC renamed +5V
- net +5V: now also C16.1, F1.2, FB3.2, JP11.1 (A), JP14.1 (A), U1.5 (VCC), U2.5 (VP), U5.1 (IN), U5.3 (EN)
- new net: F1.1, ZD1.1 (K)
- new net: R18.2, RES1.1, U8.26 (RUN)
- new net: FB3.1, USB2.A4 (VBUS), USB2.A9 (VBUS), USB2.B4 (VBUS), USB2.B9 (VBUS)
- new net: R7.2, USB1.A5 (CC1)
- new net: FB4.1, USB1.A4 (VBUS), USB1.A9 (VBUS), USB1.B4 (VBUS), USB1.B9 (VBUS)
- new net: R8.1, USB1.B5 (CC2)
- new net: R13.2, R14.1, U7.1 (~{CS}), U8.56 (QSPI_SS)
- new net: BOOT1.1, R14.2
- new net: C19.1, U8.20 (XIN), Y1.1
- new net: D36.2 (A), ENC1.S2
- new net: JP17.2 (C), R12.1
- new net: R15.1, U8.21 (XOUT)
- new net: C20.1, R15.2, Y1.3
- new net: U7.7 (IO3), U8.51 (QSPI_SD3)
- new net: U7.6 (CLK), U8.52 (QSPI_SCLK)
- new net: U7.5 (DI(IO0)), U8.53 (QSPI_SD0)
- new net: U7.3 (IO2), U8.54 (QSPI_SD2)
- new net: U7.2 (DO(IO1)), U8.55 (QSPI_SD1)
- new net: R10.2, R11.1
- new net +1V1: C13.1, C14.1, C15.1, U8.23 (DVDD), U8.45 (VREG_VOUT), U8.50 (DVDD)
- new net +3V3: C10.1, C11.1, C12.1, C17.1, C18.1, C7.1, C8.1, C9.1, JP17.3 (B), R13.1, R18.1, U5.5 (OUT), U7.8 (VCC), U8.1 (IOVDD), U8.10 (IOVDD), U8.22 (IOVDD), U8.33 (IOVDD), U8.42 (IOVDD), U8.43 (ADC_AVDD), U8.44 (VREG_IN), U8.48 (USB_VDD), U8.49 (IOVDD)
- new net D+: R16.2, U6.1 (IO1), U6.6 (IO4), USB1.A6 (D+), USB1.B6 (D+)
- new net D-: R17.2, U6.3 (IO2), U6.4 (IO3), USB1.A7 (D-), USB1.B7 (D-)
- new net DN: R17.1, U8.46 (USB_DM)
- new net DP: R16.1, U8.47 (USB_DP)
- new net HAND: R12.2, U8.29 (GPIO18)
- new net Row5: D29.1 (K), D30.1 (K), D31.1 (K), D32.1 (K), D33.1 (K), D34.1 (K), D35.1 (K), U8.32 (GPIO21)
- new net SER+: U2.3 (IO2), U2.4 (IO3), U8.2 (GPIO0), USB2.A7 (D-), USB2.B7 (D-)
- new net SER-: U2.1 (IO1), U2.6 (IO4), U8.3 (GPIO1), USB2.A6 (D+), USB2.B6 (D+)
- new net VBUS: FB4.2, R9.1, U6.5 (VP), ZD1.2 (A)
- new net VBUS_DETECT: R10.1, R9.2, U8.30 (GPIO19)
- no-connect marks 13 -> 18
Other:
- note added: "DO NOT CHANGE!"
- note added: "Power"
- company: (none) -> Tweety's Wild Thinking
- title: (none) -> RefleXion - X65
- moved on the sheet: D1, D10, D11, D12, D13, D14, D15, D16, D17, D18, D19, D2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
