File: RefleXion 65/RefleXion 65 - Front Plate Module/RefleXion - 65 Front Plate Module.kicad_pcb (KiCad board)
At the start: 2 copper layers, 133.4 x 122.1 mm, 44 parts, among them SW1 SW_Push, SW10 SW_Push, SW11 SW_Push, SW12 SW_Push, SW13 SW_Push, SW14 SW_Push, SW15 SW_Push, SW16 SW_Push, SW17 SW_Push, SW18 SW_Push, SW19 SW_Push, SW2 SW_Push, SW20 SW_Push, SW21 SW_Push, SW22 SW_Push, SW23 SW_Push, SW24 SW_Push, SW25 SW_Push, SW26 SW_Push, SW27 SW_Push, SW28 SW_Push, SW29 SW_Push, SW3 SW_Push, SW30 SW_Push, SW31 SW_Push, SW32 SW_Push, SW33 SW_Push, SW4 SW_Push, SW5 SW_Push, SW6 SW_Push, SW7 SW_Push, SW8 SW_Push, SW9 SW_Push

Commit message: X65 initial commit
Parts:
- removed H5, H6: Spacer_Plate, Keyboard_Plate:Spacer Plate hole
- ENC3: footprint Keyboard Encoders:Encoder_Plate_Placeholder -> Keyboard Encoders:Encoder_Plate_Placeholder_nodrill
- ST1: footprint Keyboard_Plate:Stabilizer_Cherry_MX_2.00u_PLate -> Keyboard_Plate:Stabilizer_Plate_2_to_1
- SW1, SW10, SW11, SW12, SW13, SW14, SW15, SW16, SW17, SW18, SW19, SW2, SW20, SW21, SW22, SW23, SW24, SW25, SW26, SW27, SW28, SW29, SW3, SW30, SW31, SW32, SW33, SW4, SW5, SW6, SW7, SW8, SW9: footprint Keyboard_Plate:SW_MX_Plate_Placeholder -> Keyboard_Plate:SW_MX_Plate_Placeholder_nodrill
- moved ENC3 2.00 mm to (84.1, 25.6)
- moved OLED1 2.00 mm to (126.1, 25.6)
- moved G*** 1.50 mm to (101.1, 25.6)
- moved G*** 1.50 mm to (101.0, 25.0)
