File: RefleXion X65/PCB/RefleXion X65.kicad_pcb (KiCad board)
At the start: 2 copper layers, 133.4 x 117.1 mm, 169 parts, among them SW1 SW_Push, SW10 SW_Push, SW11 SW_Push, SW12 SW_Push, SW13 SW_Push, SW14 SW_Push, SW15 SW_Push, SW16 SW_Push, SW17 SW_Push, SW18 SW_Push, SW19 SW_Push, SW2 SW_Push, SW20 SW_Push, SW21 SW_Push, SW22 SW_Push, SW23 SW_Push, SW24 SW_Push, SW25 SW_Push, SW26 SW_Push, SW27 SW_Push, SW28 SW_Push, SW29 SW_Push, SW3 SW_Push, SW30 SW_Push, SW31 SW_Push, SW32 SW_Push, SW33 SW_Push, SW34 SW_Push, SW35 SW_Push, SW36 SW_Push, SW4 SW_Push, SW5 SW_Push, SW6 SW_Push, SW7 SW_Push, SW8 SW_Push, SW9 SW_Push, U1 SN74LV1T34DBV, U2 SRV05-4, U5 SPX3819M5-L-3-3/TR, U6 SRV05-4, U7 W25Q32JVUUIQ, U8 RP2040, Y1 TXM12M0004252LBCEO00T

Commit message: v1.10 test1
Parts:
- removed JP10, JP11, JP12, JP13, JP14, JP15, JP16, JP9: Jumper_2_Open, Keyboard Common:Jumper_min_v2
- JP17: moved to F.Cu
- OLED1: footprint Keyboard Common:SSD1306-0.91-OLED-4pin-128x32 -> Keyboard Common:SSD1306-0.91-OLED-4pin-128x32 doublesided
- moved JP17 46.4 mm to (97.8, 22.9), turned to 0 degrees
- moved U1 43.5 mm to (71.2, 38.0), turned to 0 degrees
- moved R9 42.4 mm to (90.7, 22.9), turned to -90 degrees
- moved R11 40.7 mm to (92.6, 22.9), turned to -90 degrees
- moved R10 40.6 mm to (91.7, 22.9), turned to 90 degrees
- moved C17 36.2 mm to (94.6, 24.2), turned to 180 degrees
- moved R12 35.6 mm to (98.4, 24.9)
- moved C20 33.2 mm to (102.4, 23.6), turned to 45 degrees
- moved C19 32.7 mm to (106.1, 25.5), turned to -135 degrees
- moved Y1 32.3 mm to (104.4, 24.4), turned to -135 degrees
- moved C7 32.2 mm to (96.0, 26.5), turned to 135 degrees
- moved R15 31.3 mm to (102.8, 26.0), turned to 135 degrees
- moved C12 30.9 mm to (93.3, 29.0), turned to 135 degrees
- moved C8 30.1 mm to (103.5, 27.3), turned to 45 degrees
- moved C13 29.6 mm to (104.2, 28.0), turned to 45 degrees
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Connections:
- OLED1 pad 1: Net-(JP12-B) -> GND
- OLED1 pad 2: Net-(JP11-B) -> +3V3
- OLED1 pad 3: Net-(JP10-B) -> SCL
- OLED1 pad 4: Net-(JP13-B) -> SDA
- U8 pad 11: unconnected-(U8-GPIO8-Pad11) -> HAND
- U8 pad 13: Col6 -> unconnected-(U8-GPIO10-Pad13)
- U8 pad 14: Col5 -> unconnected-(U8-GPIO11-Pad14)
- U8 pad 15: Col4 -> unconnected-(U8-GPIO12-Pad15)
- U8 pad 16: Row0 -> unconnected-(U8-GPIO13-Pad16)
- U8 pad 2: SER+ -> Row0
- U8 pad 29: HAND -> SER+
- U8 pad 3: SER- -> Col0
- U8 pad 30: /VBUS_DETECT -> SER-
- U8 pad 31: RGB -> Col6
- U8 pad 32: Row5 -> Col5
- U8 pad 34: Row4 -> Col4
- U8 pad 35: Row3 -> Col3
- U8 pad 36: Row2 -> Row1
- U8 pad 37: Col2 -> Row2
- U8 pad 38: Col1 -> Row3
- U8 pad 39: Col0 -> Row4
- U8 pad 4: unconnected-(U8-GPIO2-Pad4) -> RGB
- U8 pad 40: Row1 -> Row5
- U8 pad 41: Col3 -> Col2
- U8 pad 5: unconnected-(U8-GPIO3-Pad5) -> Col1
- U8 pad 9: unconnected-(U8-GPIO7-Pad9) -> /VBUS_DETECT
Routing:
- net +5V: track 876.5 -> 945.6 mm, vias 47 -> 52
- net Row0: track 78.0 -> 13.7 mm, vias 2 -> 0
- net Net-(LED1-DIN): track 99.5 -> 37.1 mm, vias 5 -> 2
- net VBUS: track 76.1 -> 26.3 mm, vias 5 -> 2
- net Col1: track 157.5 -> 116.0 mm, vias 13 -> 12
- net Col0: track 178.4 -> 139.6 mm, vias 13 -> 11
- net Col2: track 128.6 -> 91.3 mm, vias 13 -> 10
- net EncA: track 53.6 -> 18.0 mm, vias 2 -> 1
- net EncB: track 57.8 -> 22.5 mm, vias 2 -> 1
- net GND: track 163.8 -> 132.7 mm, vias 64 -> 78
- net Col6: track 156.7 -> 184.1 mm, vias 13 -> 12
- net Col5: track 115.8 -> 139.4 mm, vias 11 -> 10
- net D-: track 49.2 -> 26.3 mm, vias 0 -> 2
- net D+: track 49.8 -> 26.9 mm, vias 2 -> 1
- net SER-: track 29.2 -> 51.7 mm, vias 0 -> 2
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
Commit message: Test Mosfet version
Parts:
- added Q1: 2n2007, Package_TO_SOT_SMD:SOT-23, B.Cu at (139.7, 125.8)
- added Q2: 2n2007, Package_TO_SOT_SMD:SOT-23, B.Cu at (140.5, 114.1)
- moved LED35 13.9 mm to (168.0, 128.7), turned to 90 degrees
- moved LED36 13.9 mm to (158.5, 118.6)
- moved D34 0.92 mm to (153.1, 114.4)
- moved D35 0.87 mm to (163.8, 114.5)
Connections:
- LED34 pad 3: GND -> Net-(LED34-GND)
- LED35 pad 2: Net-(LED35-DOUT) -> unconnected-(LED35-DOUT-Pad2)
- LED35 pad 3: GND -> Net-(LED34-GND)
- LED36 pad 3: GND -> Net-(LED36-GND)
- LED36 pad 4: Net-(LED35-DOUT) -> Net-(LED33-DOUT)
- U8 pad 15: unconnected-(U8-GPIO12-Pad15) -> SER+
- U8 pad 16: unconnected-(U8-GPIO13-Pad16) -> SER-
- U8 pad 29: SER+ -> Col6
- U8 pad 30: SER- -> Col5
- U8 pad 31: Col6 -> 2u
- U8 pad 32: Col5 -> 1u
Routing:
- net 1u: track 0.00 -> 123.3 mm
- net 2u: track 0.00 -> 112.0 mm
- net +5V: track 945.6 -> 988.4 mm, vias 52 -> 54
- net Net-(LED34-GND): track 0.00 -> 42.4 mm, vias 0 -> 3
- net Net-(LED35-DOUT): track 24.6 -> 0.00 mm, vias 2 -> 0
- net GND: track 132.7 -> 109.4 mm, vias 78 -> 84
- net Net-(LED36-GND): track 0.00 -> 23.1 mm, vias 0 -> 3
- net Net-(LED33-DOUT): track 22.2 -> 45.1 mm, vias 2 -> 3
- net Net-(LED34-DOUT): track 25.1 -> 43.8 mm, vias 3 -> 2
- net SER+: track 51.3 -> 62.7 mm
- net SER-: track 51.7 -> 62.3 mm
- net +1V1: track 20.2 -> 27.0 mm
- net RGB: track 36.5 -> 34.0 mm
- net +3V3: track 75.5 -> 77.8 mm
- net Net-(U8-RUN): track 20.5 -> 22.5 mm, vias 0 -> 2
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Other:
- board text added: "1x2u"
- board text added: "2x1u"

Commit message: Reflexion X65 v1.10
PCB finalized
Parts:
- added JP1: Jumper_2_Open, Keyboard Common:Jumper_min_v2, F.Cu at (153.1, 114.3)
- added JP2: Jumper_2_Open, Keyboard Common:Jumper_min_v2, F.Cu at (140.6, 130.8)
- added LED37: SK6812MINI-E, Keyboard RGB:MX_SK6812MINI-E_REVERSIBLE_special, F.Cu at (63.3, 57.0)
- added LED38: SK6812MINI-E, Keyboard RGB:MX_SK6812MINI-E_REVERSIBLE_special, F.Cu at (63.3, 76.1)
- added LED39: SK6812MINI-E, Keyboard RGB:MX_SK6812MINI-E_REVERSIBLE_special, F.Cu at (63.3, 95.1)
- added LED40: SK6812MINI-E, Keyboard RGB:MX_SK6812MINI-E_REVERSIBLE_special, F.Cu at (63.3, 114.2)
- added LED41: SK6812MINI-E, Keyboard RGB:MX_SK6812MINI-E_REVERSIBLE_special, F.Cu at (158.5, 112.8)
- added LED42: SK6812MINI-E, Keyboard RGB:MX_SK6812MINI-E_REVERSIBLE_special, F.Cu at (158.5, 95.1)
- added LED43: SK6812MINI-E, Keyboard RGB:MX_SK6812MINI-E_REVERSIBLE_special, F.Cu at (158.5, 76.1)
- added LED44: SK6812MINI-E, Keyboard RGB:MX_SK6812MINI-E_REVERSIBLE_special, F.Cu at (158.5, 57.0)
- moved Q1 112.1 mm to (70.7, 37.3)
- moved Q2 89.2 mm to (71.9, 57.1)
- moved JP17 24.4 mm to (119.7, 33.8), turned to 180 degrees
- moved U1 21.9 mm to (82.3, 56.9), turned to 180 degrees
- moved R10 20.8 mm to (76.5, 37.1)
- moved R11 20.8 mm to (77.4, 37.1), turned to 90 degrees
- moved R9 20.8 mm to (75.5, 37.1)
- moved ZD1 20.2 mm to (76.5, 35.1)
- moved C16 20.0 mm to (82.2, 35.8), turned to -90 degrees
- moved U5 19.2 mm to (84.4, 36.7)
- moved F1 19.1 mm to (79.6, 34.9), turned to 0 degrees
- moved C17 18.4 mm to (82.2, 37.7), turned to 90 degrees
- moved U6 14.3 mm to (91.5, 28.9), turned to 180 degrees
- moved R13 14.1 mm to (103.8, 23.7), turned to 90 degrees
- moved C20 13.5 mm to (109.5, 35.1), turned to -45 degrees
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Connections:
- net Net-(LED1-DIN) renamed /RGB_5
- LED1 pad 3: GND -> Net-(LED1-GND)
- LED10 pad 3: GND -> Net-(LED1-GND)
- LED11 pad 3: GND -> Net-(LED1-GND)
- LED12 pad 3: GND -> Net-(LED1-GND)
- LED13 pad 3: GND -> Net-(LED1-GND)
- LED14 pad 3: GND -> Net-(LED1-GND)
- LED15 pad 3: GND -> Net-(LED1-GND)
- LED16 pad 3: GND -> Net-(LED1-GND)
- LED17 pad 3: GND -> Net-(LED1-GND)
- LED18 pad 3: GND -> Net-(LED1-GND)
- LED19 pad 3: GND -> Net-(LED1-GND)
- LED2 pad 3: GND -> Net-(LED1-GND)
- LED20 pad 3: GND -> Net-(LED1-GND)
- LED21 pad 3: GND -> Net-(LED1-GND)
- LED22 pad 3: GND -> Net-(LED1-GND)
- LED23 pad 3: GND -> Net-(LED1-GND)
- LED24 pad 3: GND -> Net-(LED1-GND)
- LED25 pad 3: GND -> Net-(LED1-GND)
- LED26 pad 3: GND -> Net-(LED1-GND)
- LED27 pad 3: GND -> Net-(LED1-GND)
- LED28 pad 3: GND -> Net-(LED1-GND)
- LED29 pad 3: GND -> Net-(LED1-GND)
- LED3 pad 3: GND -> Net-(LED1-GND)
- LED30 pad 3: GND -> Net-(LED1-GND)
- LED31 pad 3: GND -> Net-(LED1-GND)
- LED32 pad 3: GND -> Net-(LED1-GND)
- LED33 pad 3: GND -> Net-(LED1-GND)
- LED34 pad 1: +5V -> Net-(JP2-B)
- LED34 pad 3: Net-(LED34-GND) -> Net-(LED1-GND)
- LED35 pad 1: +5V -> Net-(JP2-B)
- LED35 pad 3: Net-(LED34-GND) -> Net-(LED1-GND)
- LED36 pad 1: +5V -> Net-(JP1-B)
- LED36 pad 3: Net-(LED36-GND) -> Net-(LED1-GND)
- LED4 pad 3: GND -> Net-(LED1-GND)
- LED5 pad 3: GND -> Net-(LED1-GND)
- LED6 pad 3: GND -> Net-(LED1-GND)
- LED7 pad 3: GND -> Net-(LED1-GND)
- LED8 pad 3: GND -> Net-(LED1-GND)
- LED9 pad 3: GND -> Net-(LED1-GND)
- Q1 pad 1: 1u -> KEY
- Q1 pad 3: Net-(LED34-GND) -> Net-(LED1-GND)
- Q2 pad 1: 2u -> GLOW
- Q2 pad 3: Net-(LED36-GND) -> Net-(LED37-GND)
- R10 pad 1: /VBUS_DETECT -> VBUS_DETECT
- R9 pad 2: /VBUS_DETECT -> VBUS_DETECT
- U1 pad 2: RGB -> RGB_3
- U8 pad 11: HAND -> unconnected-(U8-GPIO8-Pad11)
- U8 pad 12: unconnected-(U8-GPIO9-Pad12) -> SER+
- U8 pad 13: unconnected-(U8-GPIO10-Pad13) -> SER-
- U8 pad 14: unconnected-(U8-GPIO11-Pad14) -> HAND
- U8 pad 15: SER+ -> Col6
- U8 pad 16: SER- -> Col5
- U8 pad 17: unconnected-(U8-GPIO14-Pad17) -> Col4
- U8 pad 18: unconnected-(U8-GPIO15-Pad18) -> Col3
- U8 pad 2: Row0 -> unconnected-(U8-GPIO0-Pad2)
- U8 pad 27: SDA -> unconnected-(U8-GPIO16-Pad27)
- U8 pad 28: SCL -> GLOW
- U8 pad 29: Col6 -> KEY
- U8 pad 3: Col0 -> EncB
- U8 pad 30: Col5 -> Row1
- U8 pad 31: 2u -> Row2
- U8 pad 32: 1u -> Row3
- U8 pad 34: Col4 -> Row4
- U8 pad 35: Col3 -> Row5
- U8 pad 36: Row1 -> Col2
- U8 pad 37: Row2 -> RGB_3
- U8 pad 38: Row3 -> Col0
- U8 pad 39: Row4 -> VBUS_DETECT
- U8 pad 4: RGB -> EncA
- U8 pad 40: Row5 -> Col1
- U8 pad 41: Col2 -> Row0
- U8 pad 5: Col1 -> unconnected-(U8-GPIO3-Pad5)
- U8 pad 6: unconnected-(U8-GPIO4-Pad6) -> SDA
- U8 pad 7: EncB -> SCL
- U8 pad 8: EncA -> unconnected-(U8-GPIO6-Pad8)
- U8 pad 9: /VBUS_DETECT -> unconnected-(U8-GPIO7-Pad9)
Routing:
- net Net-(LED1-GND): track 0.00 -> 816.8 mm, vias 0 -> 43
- net Net-(LED37-GND): track 0.00 -> 237.2 mm, vias 0 -> 14
- net 1u: track 123.3 -> 0.00 mm
- net Net-(LED40-DOUT): track 0.00 -> 112.2 mm, vias 0 -> 2
- net 2u: track 112.0 -> 0.00 mm
- net GND: track 109.4 -> 34.2 mm, vias 84 -> 56
- net +5V: track 988.4 -> 920.2 mm, vias 54 -> 62
- net GLOW: track 0.00 -> 49.2 mm, vias 0 -> 4
- net Net-(LED34-GND): track 42.4 -> 0.00 mm, vias 3 -> 0
- net KEY: track 0.00 -> 36.1 mm, vias 0 -> 2
- net RGB: track 34.0 -> 0.00 mm, vias 2 -> 0
- net Net-(JP2-B): track 0.00 -> 31.8 mm, vias 0 -> 2
- net Net-(LED42-DOUT): track 0.00 -> 30.2 mm, vias 0 -> 3
- net RGB_3: track 0.00 -> 29.7 mm
- net Net-(LED43-DOUT): track 0.00 -> 29.1 mm, vias 0 -> 3
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Other:
- board text added: "Close jumpers for OLED on LEFT Hand"
- board text added: "Close jumpers for OLED on RIGHT Hand"
- board text removed: "Close for OLED on LEFT Hand"
- board text removed: "Close for OLED on RIGHT Hand"
