File: RefleXion Grid/RefleXion Grid - PCB/RefleXion Grid.kicad_pcb (KiCad board)
At the start: 2 copper layers, 152.4 x 102.7 mm, 215 parts, among them J1 USB_C_Receptacle_USB2.0, J2 USB_C_Receptacle_USB2.0, SW1 SW_Push, SW10 SW_Push, SW11 SW_Push, SW12 SW_Push, SW13 SW_Push, SW14 SW_Push, SW15 SW_Push, SW16 SW_Push, SW17 SW_Push, SW18 SW_Push, SW19 SW_Push, SW2 SW_Push, SW20 SW_Push, SW21 SW_Push, SW22 SW_Push, SW23 SW_Push, SW24 SW_Push, SW24A1 SW_Push, SW25 SW_Push, SW25A1 SW_Push, SW26 SW_Push, SW27 SW_Push, SW28 SW_Push, SW29 SW_Push, SW3 SW_Push, SW30 SW_Push, SW31 SW_Push, SW32 SW_Push, SW33 SW_Push, SW33A1 SW_Push, SW34 SW_Push, SW35 SW_Push, SW36 SW_Push, SW37 SW_Push, SW38 SW_Push, SW39 SW_Push, SW4 SW_Push, SW40 SW_Push, SW5 SW_Push, SW6 SW_Push, SW7 SW_Push, SW8 SW_Push, SW9 SW_Push, U1 W25Q32JVUUIQ, U2 RP2040, U3 SRV05-4, U4 SPX3819M5-L-3-3/TR, U6 SN74LV1T34DBV, Y1 TXM12M0004252LBCEO00T

Commit message: in progress grid
Parts:
- removed BOOT1: YTSA010, Keyboard Common:YTS-A002
- removed C19, C3, C4, C7, C8: 100nF, Capacitor_SMD:C_0402_1005Metric
- removed D15, D23, D31, D39, D7: 1N4148W, Diode_SMD:D_SOD-123
- removed ENC1, ENC10, ENC11, ENC12, ENC2, ENC3, ENC4, ENC5, ENC6, ENC7, ENC8, ENC9: Rotary_Encoder_Click, Keyboard Encoders:Encoder_Alps_EC11E_Small
- removed H5: Spacer_PCB, Keyboard Common:Spacer PCB hole
- removed JP14: Jumper_2_Open, Keyboard Common:Jumper_min_v2
- removed LED15, LED23, LED31, LED7: SK6812MINI-E, Keyboard RGB:MX_SK6812MINI-E_REVERSIBLE
- removed LED25A1, LED33A1, LED39: SK6812MINI-E, Keyboard RGB:MX_SK6812MINI-E_REVERSIBLE_special
- removed R2: 1K, Resistor_SMD:R_0402_1005Metric
- removed ST3: Stabilizer_2u_MX, Keyboard Stabilizer:Stabilizer_Cherry_MX_2.00u
- removed SW15, SW23, SW25A1, SW31, SW33A1, SW39, SW7: SW_Push, Keyboard Switches:SW_MX_HotSwap_Reversible
- added FB2: BLM18SG700TZ1D, Capacitor_SMD:C_0603_1608Metric_Pad1.08x0.95mm_HandSolder, B.Cu at (72.6, 39.0)
- added FB3: BLM18SG700TZ1D, Capacitor_SMD:C_0603_1608Metric_Pad1.08x0.95mm_HandSolder, B.Cu at (107.0, 32.7)
- added H4: Spacer_PCB, Keyboard Common:Spacer PCB hole, F.Cu at (88.7, 114.6)
- added H8: Spacer_PCB, Keyboard Common:Spacer PCB hole, F.Cu at (183.9, 114.6)
- added H9: Spacer_PCB, Keyboard Common:Spacer PCB hole, F.Cu at (164.9, 114.6)
- added JP20: Jumper_2_Open, Keyboard Common:Jumper_min_v2, F.Cu at (79.1, 74.4)
- added LED32A1: SK6812MINI-E, Keyboard RGB:MX_SK6812MINI-E_REVERSIBLE_SMALL_PAD, F.Cu at (88.7, 129.1)
- added RES2: YTSA010, Keyboard Common:YTS-A002, F.Cu at (70.8, 53.6)
- added SW32A1: SW_Push, Keyboard Switches:SW_MX_HotSwap_Reversible, F.Cu at (88.7, 124.1)
- LED1, LED10, LED11, LED12, LED13, LED14, LED17, LED18, LED19, LED2, LED20, LED21, LED22, LED28, LED29, LED3, LED30, LED32, LED36, LED4, LED44, LED45, LED46, LED5, LED6, LED9: footprint Keyboard RGB:MX_SK6812MINI-E_REVERSIBLE -> Keyboard RGB:MX_SK6812MINI-E_REVERSIBLE_SMALL_PAD
- LED16, LED24, LED24A1, LED25, LED26, LED27, LED33, LED34, LED35, LED37, LED38, LED40, LED8: footprint Keyboard RGB:MX_SK6812MINI-E_REVERSIBLE_special -> Keyboard RGB:MX_SK6812MINI-E_REVERSIBLE_SMALL_PAD
- SW29, SW30, SW37, SW38, SW5, SW6: footprint Keyboard Switches:SW_MX_HotSwap_Reversible -> Keyboard Switches:SW_MX_HotSwap_Reversible_Encoder
- U2: footprint Package_DFN_QFN:QFN-56-1EP_7x7mm_P0.4mm_EP3.2x3.2mm -> Package_DFN_QFN:QFN-56-1EP_7x7mm_P0.4mm_EP3.2x3.2mm_ThermalVias
- moved JP19 122.3 mm to (79.1, 55.4), turned to 0 degrees
- moved D32 19.0 mm to (106.7, 126.4)
- moved D33 19.0 mm to (109.0, 126.4)
- moved ST1 19.0 mm to (88.7, 105.0)
- moved ST2 19.0 mm to (88.7, 124.1)
- moved D25 17.2 mm to (94.7, 95.5)
- moved D26 17.0 mm to (108.6, 107.3)
- moved D6 16.4 mm to (182.6, 50.0), turned to 90 degrees
- moved D22 16.3 mm to (182.6, 88.7), turned to 90 degrees
- moved D5 16.3 mm to (163.6, 49.9), turned to 90 degrees
- moved D21 16.0 mm to (163.6, 88.3), turned to 90 degrees
- moved D37 14.7 mm to (163.6, 125.4), turned to 90 degrees
- moved D38 14.5 mm to (182.7, 125.2), turned to 90 degrees
- moved H3 14.1 mm to (183.9, 35.9)
- moved H7 14.0 mm to (183.9, 95.5)
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Connections:
- net Enc1 renamed Net-(D5-A)
- net Enc10 renamed Net-(D8-A)
- net Enc11 renamed Net-(D16-A)
- net Enc12 renamed Net-(D32-A)
- net Enc2 renamed Net-(D6-A)
- net Enc4 renamed Net-(D29-A)
- net Enc5 renamed Net-(D30-A)
- net Enc7 renamed Net-(D37-A)
- net Enc8 renamed Net-(D38-A)
- J1 pad S1: GND -> Earth_Protective
- J2 pad S1: GND -> Earth_Protective
- LED1 pad 4: Net-(LED1-DIN) -> Net-(JP19-B)
- LED14 pad 4: Net-(JP14-A) -> Net-(LED14-DIN)
- LED22 pad 2: Net-(JP19-B) -> Net-(LED22-DOUT)
- LED24A1 pad 2: Net-(LED24-DIN) -> Net-(LED24A1-DOUT)
- LED24A1 pad 4: Net-(LED24A1-DIN) -> Net-(LED24-DOUT)
- LED25 pad 2: Net-(LED24A1-DIN) -> Net-(LED24-DIN)
- LED25 pad 4: Net-(LED25-DIN) -> Net-(LED24A1-DOUT)
- LED26 pad 2: Net-(LED25A1-DIN) -> Net-(LED24A1-DOUT)
- LED30 pad 4: Net-(JP19-A) -> Net-(LED22-DOUT)
- LED33 pad 2: Net-(LED33-DOUT) -> Net-(LED32A1-DOUT)
- LED34 pad 4: Net-(LED33A1-DOUT) -> Net-(LED32A1-DOUT)
- LED38 pad 2: Net-(LED38-DOUT) -> unconnected-(LED38-DOUT-Pad2)_1
- LED40 pad 2: Net-(LED1-DIN) -> Net-(JP19-B)
- LED40 pad 4: Net-(LED40-DIN) -> Net-(JP19-A)
- LED46 pad 2: Net-(LED40-DIN) -> Net-(JP19-A)
- LED6 pad 2: Net-(JP14-B) -> Net-(LED14-DIN)
- RES1 pad 3: GND -> Earth_Protective
- SW24A1 pad 1: Net-(D24-A) -> Col0
- SW24A1 pad 2: Col0 -> Net-(D24-A)
- U2 pad 12: Col3 -> Row2
- U2 pad 16: Row1 -> unconnected-(U2-GPIO13-Pad16)
- U2 pad 17: Row2 -> Col3
- U2 pad 35: EncD -> unconnected-(U2-GPIO23-Pad35)
- U2 pad 36: EncC -> unconnected-(U2-GPIO24-Pad36)
- U2 pad 4: Col7 -> Col6
- U2 pad 5: Col6 -> Col5
- U2 pad 6: Col5 -> EncA
- U2 pad 7: EncA -> EncB
- U2 pad 8: EncB -> Col4
- U2 pad 9: Col4 -> Row1
Routing:
- net GND: track 435.1 -> 1000.5 mm, vias 252 -> 70
- net EncC: track 351.5 -> 0.00 mm, vias 7 -> 0
- net Col7: track 234.6 -> 0.00 mm, vias 11 -> 0
- net +5V: track 1054.1 -> 861.6 mm, vias 77 -> 51
- net EncA: track 133.1 -> 245.7 mm, vias 3 -> 4
- net Net-(LED40-DIN): track 102.1 -> 0.00 mm, vias 6 -> 0
- net EncB: track 354.0 -> 254.0 mm, vias 5 -> 3
- net EncD: track 98.5 -> 0.00 mm, vias 3 -> 0
- net Row4: track 261.5 -> 170.9 mm, vias 11 -> 7
- net Row0: track 178.3 -> 112.6 mm, vias 5 -> 7
- net Net-(LED24A1-DIN): track 61.4 -> 0.00 mm, vias 5 -> 0
- net Net-(JP19-A): track 35.5 -> 92.5 mm, vias 2 -> 4
- net Net-(LED33-DOUT): track 45.5 -> 0.00 mm, vias 3 -> 0
- net Row3: track 216.4 -> 173.1 mm, vias 6 -> 8
- net Row2: track 176.7 -> 134.8 mm, vias 4 -> 7
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- added copper zone on B.Cu, net Earth_Protective
- added copper zone on F.Cu, net Earth_Protective
- removed copper zone on B.Cu, net GND
- removed copper zone on F.Cu, net GND
Other:
- board size 152.4 x 102.7 mm -> 133.4 x 102.7 mm
- board text added: "RGB bypass"
- board text removed: "Bypass for RGB when breaking off columns."
