File: RefleXion Grid/RefleXion Grid - PCB/RefleXion Grid.kicad_sch (KiCad schematic)
At the start: 215 parts, among them J1 USB_C_Receptacle_USB2.0, J2 USB_C_Receptacle_USB2.0, SW1 SW_Push, SW10 SW_Push, SW11 SW_Push, SW12 SW_Push, SW13 SW_Push, SW14 SW_Push, SW15 SW_Push, SW16 SW_Push, SW17 SW_Push, SW18 SW_Push, SW19 SW_Push, SW2 SW_Push, SW20 SW_Push, SW21 SW_Push, SW22 SW_Push, SW23 SW_Push, SW24 SW_Push, SW24A1 SW_Push, SW25 SW_Push, SW25A1 SW_Push, SW26 SW_Push, SW27 SW_Push, SW28 SW_Push, SW29 SW_Push, SW3 SW_Push, SW30 SW_Push, SW31 SW_Push, SW32 SW_Push, SW33 SW_Push, SW33A1 SW_Push, SW34 SW_Push, SW35 SW_Push, SW36 SW_Push, SW37 SW_Push, SW38 SW_Push, SW39 SW_Push, SW4 SW_Push, SW40 SW_Push, SW5 SW_Push, SW6 SW_Push, SW7 SW_Push, SW8 SW_Push, SW9 SW_Push, U1 W25Q32JVUUIQ, U2 RP2040, U3 SRV05-4, U4 SPX3819M5-L-3-3/TR, U6 SN74LV1T34DBV, Y1 TXM12M0004252LBCEO00T

Commit message: in progress grid
Parts:
- removed BOOT1: YTSA010, Keyboard Common:YTS-A002, symbol Keyboard Common:TS-A002
- removed C19: 100nF, Capacitor_SMD:C_0402_1005Metric, symbol Device:C
- removed C3, C4, C7, C8: 100nF, Capacitor_SMD:C_0402_1005Metric, symbol Device:C_Small
- removed D15, D23, D31, D39, D7: 1N4148W, Diode_SMD:D_SOD-123, symbol Diode:1N4148W
- removed ENC1, ENC10, ENC11, ENC12, ENC2, ENC3, ENC4, ENC5, ENC6, ENC7, ENC8, ENC9: Rotary_Encoder_Click, Keyboard Encoders:Encoder_Alps_EC11E_Small, symbol Keyboard Switches:Rotary_Encoder_Click
- removed H5: Spacer_PCB, Keyboard Common:Spacer PCB hole, symbol Keyboard_Plate:Spacer_PCB
- removed JP14: Jumper_2_Open, Keyboard Common:Jumper_min_v2, symbol Jumper:Jumper_2_Open
- removed LED15, LED23, LED31, LED7: SK6812MINI-E, Keyboard RGB:MX_SK6812MINI-E_REVERSIBLE, symbol Keyboard Common:SK6812MINI-E
- removed LED25A1, LED33A1, LED39: SK6812MINI-E, Keyboard RGB:MX_SK6812MINI-E_REVERSIBLE_special, symbol Keyboard Common:SK6812MINI-E
- removed R2: 1K, Resistor_SMD:R_0402_1005Metric, symbol Device:R
- removed ST3: Stabilizer_2u_MX, Keyboard Stabilizer:Stabilizer_Cherry_MX_2.00u, symbol Keyboard Switches:Stabilizer_2u_MX
- removed SW15, SW23, SW25A1, SW31, SW33A1, SW39, SW7: SW_Push, Keyboard Switches:SW_MX_HotSwap_Reversible, symbol Keyboard Switches:SW_MX_HotSwap_Reversible
- added FB2, FB3: BLM18SG700TZ1D, Capacitor_SMD:C_0603_1608Metric_Pad1.08x0.95mm_HandSolder, symbol LCSC Parts:Ferrite Bead
- added H8, H9: Spacer_PCB, Keyboard Common:Spacer PCB hole, symbol Keyboard_Plate:Spacer_PCB
- added JP20: Jumper_2_Open, Keyboard Common:Jumper_min_v2, symbol Jumper:Jumper_2_Open
- added LED32A1: SK6812MINI-E, Keyboard RGB:MX_SK6812MINI-E_REVERSIBLE_SMALL_PAD, symbol Keyboard Common:SK6812MINI-E
- added RES2: YTSA010, Keyboard Common:YTS-A002, symbol Keyboard Common:TS-A002
- added unit 2 of SW29
- added unit 2 of SW30
- added SW32A1: SW_Push, Keyboard Switches:SW_MX_HotSwap_Reversible, symbol Keyboard Switches:SW_MX_HotSwap_Reversible
- added unit 2 of SW37
- added unit 2 of SW38
- added unit 2 of SW5
- added unit 2 of SW6
- LED1, LED10, LED11, LED12, LED13, LED14, LED17, LED18, LED19, LED2, LED20, LED21, LED22, LED28, LED29, LED3, LED30, LED32, LED36, LED4, LED44, LED45, LED46, LED5, LED6, LED9: footprint Keyboard RGB:MX_SK6812MINI-E_REVERSIBLE -> Keyboard RGB:MX_SK6812MINI-E_REVERSIBLE_SMALL_PAD
- LED16, LED24, LED24A1, LED25, LED26, LED27, LED33, LED34, LED35, LED37, LED38, LED40, LED8: footprint Keyboard RGB:MX_SK6812MINI-E_REVERSIBLE_special -> Keyboard RGB:MX_SK6812MINI-E_REVERSIBLE_SMALL_PAD
- SW29, SW30, SW37, SW38, SW5, SW6: footprint Keyboard Switches:SW_MX_HotSwap_Reversible -> Keyboard Switches:SW_MX_HotSwap_Reversible_Encoder; symbol Keyboard Switches:SW_MX_HotSwap_Reversible -> Keyboard Switches:SW_MX_HotSwap_Reversible_Encoder
- U2: footprint Package_DFN_QFN:QFN-56-1EP_7x7mm_P0.4mm_EP3.2x3.2mm -> Package_DFN_QFN:QFN-56-1EP_7x7mm_P0.4mm_EP3.2x3.2mm_ThermalVias
Connections:
- net Col7 is gone; now on net Col6: U2.4 (GPIO2)
- net +5V: now also LED32A1.1 (VDD)
- net Col0: now also SW24A1.1, SW32A1.1; no longer SW24A1.2
- net Col3: now also U2.17 (GPIO14); no longer U2.12 (GPIO9)
- net Col4: now also U2.8 (GPIO6); no longer U2.9 (GPIO7)
- net Col5: now also U2.5 (GPIO3); no longer U2.6 (GPIO4)
- net Col6: no longer U2.5 (GPIO3)
- net Earth_Protective: now also J1.S1 (SHIELD), J2.S1 (SHIELD), RES1.3, FB2.1, FB3.1, RES2.3, SW29.MP, SW30.MP, SW37.MP, SW38.MP, SW5.MP, SW6.MP
- net EncA: now also U2.6 (GPIO4), SW29.A, SW30.A, SW37.A, SW38.A, SW5.A, SW6.A; no longer U2.7 (GPIO5)
- net EncB: now also U2.7 (GPIO5), SW29.B, SW30.B, SW37.B, SW38.B, SW5.B, SW6.B; no longer U2.8 (GPIO6)
- net GND: now also FB2.2, FB3.2, LED32A1.3 (GND), RES2.2, SW29.C, SW30.C, SW37.C, SW38.C, SW5.C, SW6.C; no longer J1.S1 (SHIELD), J2.S1 (SHIELD), RES1.3
- net Row1: now also U2.9 (GPIO7); no longer U2.16 (GPIO13)
- net Row2: now also U2.12 (GPIO9); no longer U2.17 (GPIO14)
- net at LED24.2 (DOUT), LED32.4 (DIN): now also LED24A1.4 (DIN), LED32A1.4 (DIN)
- net at LED30.4 (DIN): now also LED22.2 (DOUT); no longer JP19.1 (A)
- net at JP19.2 (B): now also LED1.4 (DIN), LED40.2 (DOUT); no longer LED22.2 (DOUT)
- net at LED14.4 (DIN): now also LED6.2 (DOUT)
- net at LED16.4 (DIN), LED8.2 (DOUT): now also JP20.1 (A)
- net at LED8.4 (DIN), LED9.2 (DOUT): now also JP20.2 (B)
- net at LED33.2 (DOUT): now also LED34.4 (DIN), LED32A1.2 (DOUT)
- net at D24.2 (A), SW24.2: now also SW24A1.2; no longer SW24A1.1
- net at R1.2, RES1.2, U2.26 (RUN): now also RES2.1
- net at LED40.4 (DIN), LED46.2 (DOUT): now also JP19.1 (A)
- net at LED24A1.2 (DOUT): now also LED25.4 (DIN), LED26.2 (DOUT); no longer LED24.4 (DIN)
- net at LED25.2 (DOUT): now also LED24.4 (DIN); no longer LED24A1.4 (DIN)
- net Enc1: no longer names the net of D5.2 (A), SW5.1
- net Enc10: no longer names the net of D8.2 (A), SW8.2
- net Enc11: no longer names the net of D16.2 (A), SW16.2
- net Enc12: no longer names the net of D32.2 (A), SW32.2
- net Enc12: now also SW32A1.2
- net Enc2: no longer names the net of D6.2 (A), SW6.1
- net Enc4: no longer names the net of D29.2 (A), SW29.1
- net Enc5: no longer names the net of D30.2 (A), SW30.1
- net Enc7: no longer names the net of D37.2 (A), SW37.1
- net Enc8: no longer names the net of D38.2 (A), SW38.1
- net EncC: no longer names the net of U2.36 (GPIO24)
- net EncD: no longer names the net of U2.35 (GPIO23)
- no-connect marks 16 -> 19
Other:
- moved on the sheet: C1, C2, C20, D1, D10, D11, D12, D13, D14, D17, D18, D19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
